File: PCB/LED2/LED.kicad_pcb (KiCad board)
At the start: 2 copper layers, 70 x 70 mm, 34 parts, among them J1 Conn_01x03, J2 USB-C, U1 ESP32-PICO-MINI-02, U2 QR, U3 MD8942, U4 Barcode, U5 CH340X

Commit message: Another cap
Parts:
- added C6: 100nF, RevK:C_0402, F.Cu at (118.3, 53.2)
Routing:
- net +3V3: track 83.6 -> 84.9 mm

Commit message: V Cuts
Other:
- board text added: "2 Designs, 0.8mm, Black"
- board text removed: "2 Designs, 0.8mm, Black, V-Cuts"

Commit message: Better Rails
Parts:
- removed FID1, FID2, FID3, FID4, FID5, FID6, FID7, FID8: Fiducial, Fiducial:Fiducial_1mm_Mask2mm
- added PCB1: 70x70, RevK:PCB7070, F.Cu at (135.0, 65.0)
Routing:
- net GND: vias 5 -> 7
Other:
- outline, holes or cut-outs redrawn

Commit message: Ordered
Parts:
- moved R2 1.91 mm to (122.8, 56.0), turned to -90 degrees
Connections:
- R2 pad 2: +3V3 -> Net-(U5-~{CTS})
- U5 pad 5: GND -> Net-(U5-~{CTS})
Routing:
- net GND: track 24.8 -> 17.4 mm, vias 7 -> 8
- net Net-(U5-~{CTS}): track 0.00 -> 2.21 mm
- net GPIO0: track 15.4 -> 14.1 mm
- net +3V3: track 84.9 -> 83.7 mm
Other:
- board text added: "RGB: 20/8/21"
- board text removed: "20/8/21"
