File: PCB/LED2/LED.kicad_sch (KiCad schematic)
At the start: 24 parts, among them J1 Conn_01x03, J2 USB-C, U1 ESP32-PICO-MINI-02, U2 QR, U3 CH340X, U5 MD8942

Commit message: As ordered
Parts:
- removed D1: LED_BARG, RevK:MHS190RGBCT, symbol Device:LED_BARG
- removed R2: 300R, RevK:R_0402, symbol Device:R
- removed R3: 1K, RevK:R_0402, symbol Device:R
- removed R4: 100R, RevK:R_0402, symbol Device:R
- added D2: RGB, RevK:LED-RGB-1.6x1.6, symbol Device:LED_RBGA
- added FID1, FID2, FID3, FID4, FID5, FID6, FID7, FID8: Fiducial, Fiducial:Fiducial_1mm_Mask2mm, symbol Mechanical:Fiducial
- added H1, H2, H3, H4: MountingHole, MountingHole:MountingHole_2mm, symbol Mechanical:MountingHole
- added R11: 2K, RevK:R_0402, symbol Device:R
- added R12: 220R, RevK:R_0402, symbol Device:R
- added R8: 680R, RevK:R_0402, symbol Device:R
- added U4, U6: Barcode, RevK:EAN-5060634238090, symbol RevK:Barcode
- D3: footprint Package_TO_SOT_SMD:SOT-23 -> RevK:SOT-23
Connections:
- net +3V3: now also D2.4 (A)
- net B: now also R12.2
- net EN: now also C1.2, R1.2, U1.8 (EN)
- net G: now also R11.2
- net R: now also R8.2
- new net: D2.2 (BK), R12.1
- new net: D2.1 (RK), R8.1
- new net: D2.3 (GK), R11.1
Other:
- moved on the sheet: R1

Commit message: Re panel
Parts:
- removed H1, H2, H3, H4: MountingHole, MountingHole:MountingHole_2mm, symbol Mechanical:MountingHole
- removed U6: Barcode, RevK:EAN-5060634238090, symbol RevK:Barcode
Other:
- moved on the sheet: FID1, FID2, FID3, FID4, FID5, FID6, FID7, FID8

Commit message: Another cap
Parts:
- added C4: 100nF, RevK:C_0402, symbol Device:C
- added R2: 4k7, RevK:R_0402, symbol Device:R
Connections:
- net +3V3: now also C4.1, R2.2
- net GND: now also C4.2
- net GPIO0: now also R2.1
Changed lines of the file:
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@@
   (junction (at 227.965 24.765) (diameter 0) (color 0 0 0 0)
+  )
+  (junction (at 247.015 46.355) (diameter 0) (color 0 0 0 0)
   )
   (junction (at 115.57 90.17) (diameter 0) (color 0 0 0 0)
@@
     (stroke (width 0) (type default))
   )
+  (wire (pts (xy 238.125 46.355) (xy 247.015 46.355))
+    (stroke (width 0) (type default))
+  )
   (wire (pts (xy 173.355 31.75) (xy 175.895 31.75))
     (stroke (width 0) (type default))
@@
   )
   (wire (pts (xy 227.965 24.765) (xy 229.235 24.765))
+    (stroke (width 0) (type default))
+  )
+  (wire (pts (xy 247.015 46.355) (xy 252.73 46.355))
     (stroke (width 0) (type default))
   )
@@
     )
   )
-  (global_label "GPIO0" (shape output) (at 238.125 46.355 0) (fields_autoplaced)
+  (global_label "GPIO0" (shape output) (at 252.73 46.355 0) (fields_autoplaced)
     (effects (font (size 1.27 1.27)) (justify left))
-    (property "Intersheetrefs" "${INTERSHEET_REFS}" (at 246.0614 46.355 0)
+    (property "Intersheetrefs" "${INTERSHEET_REFS}" (at 260.6664 46.355 0)
       (effects (font (size 1.27 1.27)) (justify left) hide)
     )
@@
         (path "/babeabf2-f3b0-4ed5-8d9e-0215947e6cf3"
           (reference "C6") (unit 1)
+        )
+      )
+    )
+  )
+  (symbol (lib_id "power:GND") (at 198.12 65.405 0) (unit 1)
+    (in_bom yes) (on_board yes) (dnp no) (fields_autoplaced)
+    (property "Reference" "#PWR0105" (at 198.12 71.755 0)
+      (effects (font (size 1.27 1.27)) hide)
+    )
+    (property "Value" "GND" (at 198.12 69.8484 0)
+      (effects (font (size 1.27 1.27)))
+    )
+    (property "Footprint" "" (at 198.12 65.405 0)
+      (effects (font (size 1.27 1.27)) hide)
+    )
+    (property "Datasheet" "" (at 198.12 65.405 0)
+      (effects (font (size 1.27 1.27)) hide)
+    )
+    (pin "1")
+    (instances
+      (project "USBA"
+        (path "/2d210a96-f81f-42a9-8bf4-1b43c11086f3"
+          (reference "#PWR0105") (unit 1)
+        )
+      )
+      (project "LED"
+        (path "/46c350bb-7de4-4e81-aafd-4af55e37aab0"
+          (reference "#PWR016") (unit 1)
         )
       )
@@
     )
   )
+  (symbol (lib_id "power:+3.3V") (at 247.015 38.735 0) (unit 1)
+    (in_bom yes) (on_board yes) (dnp no) (fields_autoplaced)
+    (property "Reference" "#PWR03" (at 247.015 42.545 0)
+      (effects (font (size 1.27 1.27)) hide)
+    )
+    (property "Value" "+3.3V" (at 247.015 35.2331 0)
+      (effects (font (size 1.27 1.27)))
+    )
+    (property "Footprint" "" (at 247.015 38.735 0)
+      (effects (font (size 1.27 1.27)) hide)
+    )
+    (property "Datasheet" "" (at 247.015 38.735 0)
+      (effects (font (size 1.27 1.27)) hide)
+    )
+    (pin "1")
+    (instances
+      (project "USBA"
+        (path "/2d210a96-f81f-42a9-8bf4-1b43c11086f3"
+          (reference "#PWR03") (unit 1)
+        )
+      )
+      (project "LED"
+        (path "/46c350bb-7de4-4e81-aafd-4af55e37aab0"
+          (reference "#PWR014") (unit 1)
+        )
+      )
+    )
+  )
   (symbol (lib_id "power:+3.3V") (at 38.1 34.925 0) (unit 1)
     (in_bom yes) (on_board yes) (dnp no)
@@
         (path "/46c350bb-7de4-4e81-aafd-4af55e37aab0"
           (reference "C1") (unit 1)
+        )
+      )
+    )
+  )
+  (symbol (lib_id "power:+3.3V") (at 198.12 57.785 0) (unit 1)
+    (in_bom yes) (on_board yes) (dnp no) (fields_autoplaced)
+    (property "Reference" "#PWR0106" (at 198.12 61.595 0)
+      (effects (font (size 1.27 1.27)) hide)
+    )
+    (property "Value" "+3.3V" (at 198.12 54.2092 0)
+      (effects (font (size 1.27 1.27)))
+    )
+    (property "Footprint" "" (at 198.12 57.785 0)
+      (effects (font (size 1.27 1.27)) hide)
+    )
+    (property "Datasheet" "" (at 198.12 57.785 0)
+      (effects (font (size 1.27 1.27)) hide)
+    )
+    (pin "1")
+    (instances
+      (project "USBA"
+        (path "/2d210a96-f81f-42a9-8bf4-1b43c11086f3"
+          (reference "#PWR0106") (unit 1)
+        )
+      )
+      (project "LED"
+        (path "/46c350bb-7de4-4e81-aafd-4af55e37aab0"
+          (reference "#PWR015") (unit 1)
         )
       )
@@
         (path "/825c70b0-4860-42b7-97dc-86bfa46e06fd"
           (reference "FID2") (unit 1)
+        )
+      )
+    )
+  )
+  (symbol (lib_id "Device:R") (at 247.015 42.545 180) (unit 1)
+    (in_bom yes) (on_board yes) (dnp no)
+    (property "Reference" "R2" (at 245.11 42.545 90)
+      (effects (font (size 1.27 1.27)))
+    )
+    (property "Value" "4k7" (at 247.015 42.545 90)
+      (effects (font (size 1.27 1.27)))
+    )
+    (property "Footprint" "RevK:R_0402" (at 248.793 42.545 90)
+      (effects (font (size 1.27 1.27)) hide)
+    )
+    (property "Datasheet" "~" (at 247.015 42.545 0)
+      (effects (font (size 1.27 1.27)) hide)
+    )
+    (pin "1")
+    (pin "2")
+    (instances
+      (project "LED"
+        (path "/46c350bb-7de4-4e81-aafd-4af55e37aab0"
+          (reference "R2") (unit 1)
         )
       )
@@
         )
       )
+    )
+  )
+  (symbol (lib_id "Device:C") (at 198.12 61.595 0) (unit 1)
+    (in_bom yes) (on_board yes) (dnp no) (fields_autoplaced)
+    (property "Reference" "C4" (at 201.041 60.7603 0)
+      (effects (font (size 1.27 1.27)) (justify left))
+    )
+    (property "Value" "100nF" (at 201.041 63.2972 0)
+      (effects (font (size 1.27 1.27)) (justify left))
+    )
+    (property "Footprint" "RevK:C_0402" (at 199.0852 65.405 0)
+      (effects (font (size 1.27 1.27)) hide)
+    )
+    (property "Datasheet" "~" (at 198.12 61.595 0)
+      (effects (font (size 1.27 1.27)) hide)
+    )
+    (pin "1")
+    (pin "2")
+    (instances
+      (project "USBA"
+        (path "/2d210a96-f81f-42a9-8bf4-1b43c11086f3"
+          (reference "C4") (unit 1)
+        )
+      )
+      (project "LED"
+        (path "/46c350bb-7de4-4e81-aafd-4af55e37aab0"
+          (reference "C6") (unit 1)
+        )
+      )

Commit message: Better Rails
Parts:
- removed FID1, FID2, FID3, FID4, FID5, FID6, FID7, FID8: Fiducial, Fiducial:Fiducial_1mm_Mask2mm, symbol Mechanical:Fiducial
- added PCB1: 70x70, RevK:PCB7070, symbol RevK:PCB

Commit message: Ordered
Connections:
- net +3V3: no longer R2.2
- net GND: no longer U3.5 (~{CTS})
- new net: R2.2, U3.5 (~{CTS})
Other:
- moved on the sheet: R2

Commit message: VCUT
Parts:
- added V1, V2: ~, RevK:VCUT70, symbol RevK:VCUT
Changed lines of the file:
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@@
+    )
+  )
+  (symbol (lib_id "RevK:VCUT") (at 259.715 176.53 0) (unit 1)
+    (in_bom yes) (on_board yes) (dnp no) (fields_autoplaced)
+    (property "Reference" "V2" (at 259.715 175.26 0)
+      (effects (font (size 1.27 1.27)) hide)
+    )
+    (property "Value" "~" (at 259.715 176.53 0)
+      (effects (font (size 1.27 1.27)))
+    )
+    (property "Footprint" "RevK:VCUT70" (at 259.715 177.8 0)
+      (effects (font (size 1.27 1.27)) hide)
+    )
+    (property "Datasheet" "" (at 259.715 176.53 0)
+      (effects (font (size 1.27 1.27)) hide)
+    )
+    (instances
+      (project "LED"
+        (path "/46c350bb-7de4-4e81-aafd-4af55e37aab0"
+          (reference "V2") (unit 1)
+        )
+      )
     )
   )
@@
       (effects (font (size 1.27 1.27)) hide)
     )
-    (property "Value" "70x70" (at 257.175 173.355 0)
+    (property "Value" "70x70" (at 256.54 173.355 0)
       (effects (font (size 1.27 1.27)) (justify left))
     )
@@
         )
       )
+    )
+  )
+  (symbol (lib_id "RevK:VCUT") (at 259.715 170.18 0) (unit 1)
+    (in_bom yes) (on_board yes) (dnp no) (fields_autoplaced)
+    (property "Reference" "V1" (at 259.715 168.91 0)
+      (effects (font (size 1.27 1.27)) hide)
+    )
+    (property "Value" "~" (at 259.715 170.18 0)
+      (effects (font (size 1.27 1.27)))
+    )
+    (property "Footprint" "RevK:VCUT70" (at 259.715 171.45 0)
+      (effects (font (size 1.27 1.27)) hide)
+    )
+    (property "Datasheet" "" (at 259.715 170.18 0)
+      (effects (font (size 1.27 1.27)) hide)
+    )
+    (instances
+      (project "LED"
+        (path "/46c350bb-7de4-4e81-aafd-4af55e37aab0"
+          (reference "V1") (unit 1)
+        )
+      )

Commit message: CH340X DTR
Parts:
- removed R2: 4k7, RevK:R_0402, symbol Device:R
- V1, V2: now left out of the parts list
Connections:
- net GPIO0: now also U3.5 (~{CTS})
Changed lines of the file:
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@@
   (junction (at 227.965 24.765) (diameter 0) (color 0 0 0 0)
   )
-  (junction (at 240.03 46.355) (diameter 0) (color 0 0 0 0)
+  (junction (at 238.125 46.355) (diameter 0) (color 0 0 0 0)
   )
   (junction (at 115.57 90.17) (diameter 0) (color 0 0 0 0)
@@
     (stroke (width 0) (type default))
   )
-  (wire (pts (xy 238.125 38.735) (xy 240.03 38.735))
-    (stroke (width 0) (type default))
-  )
   (wire (pts (xy 113.03 90.17) (xy 115.57 90.17))
     (stroke (width 0) (type default))
@@
     (stroke (width 0) (type default))
   )
+  (wire (pts (xy 238.125 38.735) (xy 238.125 46.355))
+    (stroke (width 0) (type default))
+  )
   (wire (pts (xy 73.66 59.69) (xy 77.47 59.69))
     (stroke (width 0) (type default))
@@
     (stroke (width 0) (type default))
   )
-  (wire (pts (xy 238.125 46.355) (xy 240.03 46.355))
-    (stroke (width 0) (type default))
-  )
   (wire (pts (xy 173.355 31.75) (xy 175.895 31.75))
     (stroke (width 0) (type default))
@@
     (stroke (width 0) (type default))
   )
-  (wire (pts (xy 240.03 46.355) (xy 242.57 46.355))
+  (wire (pts (xy 238.125 46.355) (xy 239.395 46.355))
     (stroke (width 0) (type default))
   )
@@
     )
   )
-  (global_label "GPIO0" (shape output) (at 242.57 46.355 0) (fields_autoplaced)
+  (global_label "GPIO0" (shape output) (at 239.395 46.355 0) (fields_autoplaced)
     (effects (font (size 1.27 1.27)) (justify left))
-    (property "Intersheetrefs" "${INTERSHEET_REFS}" (at 250.5064 46.355 0)
+    (property "Intersheetrefs" "${INTERSHEET_REFS}" (at 247.3314 46.355 0)
       (effects (font (size 1.27 1.27)) (justify left) hide)
     )
@@
     )
   )
-  (symbol (lib_id "Device:R") (at 240.03 42.545 180) (unit 1)
-    (in_bom yes) (on_board yes) (dnp no)
-    (property "Reference" "R2" (at 238.125 42.545 90)
-      (effects (font (size 1.27 1.27)))
-    )
-    (property "Value" "4k7" (at 240.03 42.545 90)
-      (effects (font (size 1.27 1.27)))
-    )
-    (property "Footprint" "RevK:R_0402" (at 241.808 42.545 90)
-      (effects (font (size 1.27 1.27)) hide)
-    )
-    (property "Datasheet" "~" (at 240.03 42.545 0)
-      (effects (font (size 1.27 1.27)) hide)
-    )
-    (pin "1")
-    (pin "2")
-    (instances
-      (project "LED"
-        (path "/46c350bb-7de4-4e81-aafd-4af55e37aab0"
-          (reference "R2") (unit 1)
-        )
-      )
-    )
-  )
   (symbol (lib_id "Connector_Generic:Conn_01x03") (at 138.43 90.17 0) (mirror x) (unit 1)
     (in_bom yes) (on_board yes) (dnp no)
@@
   )
   (symbol (lib_id "RevK:VCUT") (at 259.715 176.53 0) (unit 1)
-    (in_bom yes) (on_board yes) (dnp no) (fields_autoplaced)
+    (in_bom no) (on_board yes) (dnp no) (fields_autoplaced)
     (property "Reference" "V2" (at 259.715 175.26 0)
       (effects (font (size 1.27 1.27)) hide)
@@
     )
     (property "Datasheet" "" (at 259.715 176.53 0)
+      (effects (font (size 1.27 1.27)) hide)
+    )
+    (property "Sim.Enable" "0" (at 259.715 176.53 0)
       (effects (font (size 1.27 1.27)) hide)
     )
@@
   )
   (symbol (lib_id "RevK:VCUT") (at 259.715 170.18 0) (unit 1)
-    (in_bom yes) (on_board yes) (dnp no) (fields_autoplaced)
+    (in_bom no) (on_board yes) (dnp no) (fields_autoplaced)
     (property "Reference" "V1" (at 259.715 168.91 0)
       (effects (font (size 1.27 1.27)) hide)
@@
       (effects (font (size 1.27 1.27)) hide)
     )
+    (property "Sim.Enable" "0" (at 259.715 170.18 0)
+      (effects (font (size 1.27 1.27)) hide)
+    )

Commit message: Fix RGB
Parts:
- D2: symbol Device:LED_RBGA -> Device:LED_RGBA
Connections:
- net at R12.1: now also D2.3 (BK); no longer D2.2 (BK)
- net at R11.1: now also D2.2 (GK); no longer D2.3 (GK)
Changed lines of the file:
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@@
     )
   )
-  (symbol (lib_id "Device:LED_RBGA") (at 113.03 41.275 0) (unit 1)
+  (symbol (lib_id "Device:LED_RGBA") (at 113.03 41.275 0) (unit 1)
     (in_bom yes) (on_board yes) (dnp no)
     (property "Reference" "D2" (at 113.03 28.6512 0)
