File: PCB/150x7/150x7.kicad_pcb (KiCad board)
At the start: 2 copper layers, 14.5 x 14.5 mm, 51 parts, among them J1 Conn_01x03, J2 Conn_01x03

Commit message: Started grid
Parts:
- moved C7 13.6 mm to (109.2, 85.6), turned to 0 degrees
- moved C13 13.5 mm to (115.2, 85.6), turned to 0 degrees
- moved C14 13.4 mm to (115.2, 99.9), turned to 0 degrees
- moved C5 12.4 mm to (107.2, 85.6), turned to 0 degrees
- moved C8 11.7 mm to (109.2, 99.9), turned to 0 degrees
- moved D31 11.3 mm to (111.2, 90.8), turned to 135 degrees
- moved D5 11.3 mm to (103.2, 94.8), turned to 135 degrees
- moved D29 10.2 mm to (111.2, 86.8), turned to 135 degrees
- moved D7 10.2 mm to (103.2, 98.8), turned to 135 degrees
- moved C2 9.27 mm to (103.2, 99.9), turned to 0 degrees
- moved C11 9.16 mm to (113.2, 85.6), turned to 0 degrees
- moved D14 8.94 mm to (105.2, 98.8), turned to 135 degrees
- moved D22 8.94 mm to (109.2, 86.8), turned to 135 degrees
- moved D32 8.49 mm to (111.2, 92.8), turned to 135 degrees
- moved D4 8.49 mm to (103.2, 92.8), turned to 135 degrees
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Routing:
- net VDD: track 90.1 -> 0.00 mm, vias 6 -> 0
- net GND: track 81.3 -> 0.00 mm, vias 6 -> 0
- net Net-(D5-O): track 23.2 -> 0.00 mm, vias 2 -> 0
- net Net-(D30-O): track 22.6 -> 0.00 mm, vias 2 -> 0
- net Net-(D25-O): track 21.0 -> 0.00 mm, vias 2 -> 0
- net Net-(D10-O): track 21.0 -> 0.00 mm, vias 2 -> 0
- net Net-(D20-O): track 20.3 -> 0.00 mm, vias 2 -> 0
- net Net-(D15-O): track 20.3 -> 0.00 mm, vias 2 -> 0
- net Net-(D1-I): track 14.3 -> 0.00 mm, vias 1 -> 0
- net Net-(D35-O): track 9.11 -> 0.00 mm, vias 1 -> 0
- net Net-(D8-O): track 0.80 -> 0.00 mm
- net Net-(D7-O): track 0.80 -> 0.00 mm
- net Net-(D6-O): track 0.80 -> 0.00 mm
- net Net-(D4-O): track 0.80 -> 0.00 mm
- net Net-(D34-O): track 0.80 -> 0.00 mm
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
Commit message: Library update
Parts:
- moved D16 139.2 mm to (0.00, 0.00), turned to 0 degrees
- moved C5 25.7 mm to (107.2, 111.2)
- moved D29 24.5 mm to (111.2, 111.2), turned to 0 degrees
- moved D8 24.5 mm to (105.2, 111.2), turned to 0 degrees
- moved C11 23.7 mm to (113.2, 109.2)
- moved C13 23.7 mm to (115.2, 109.2)
- moved D22 22.5 mm to (109.2, 109.2), turned to 0 degrees
- moved C7 21.7 mm to (109.2, 107.2)
- moved D12 20.5 mm to (105.2, 115.2), turned to 0 degrees
- moved D15 20.5 mm to (107.2, 107.2), turned to 0 degrees
- moved D2 20.5 mm to (103.2, 109.2), turned to 0 degrees
- moved D24 20.5 mm to (109.2, 111.2), turned to 0 degrees
- moved D9 20.5 mm to (105.2, 109.2), turned to 0 degrees
- moved C3 19.7 mm to (105.2, 105.2)
- moved D1 18.5 mm to (103.2, 105.2), turned to 0 degrees
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Changed lines of the file:
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@@
  (footprint "RevK:SMD1010"
   (layer "F.Cu")
-  (at 107.250000 86.750000 135)
+  (at 107.250000  107.250000)
   (descr "https://cdn-shop.adafruit.com/datasheets/WS2812B.pdf")
   (tags "LED RGB NeoPixel")
@@
  (footprint "RevK:SMD1010"
   (layer "F.Cu")
-  (at 107.250000 98.750000 135)
+  (at 107.250000  113.250000)
   (descr "https://cdn-shop.adafruit.com/datasheets/WS2812B.pdf")
   (tags "LED RGB NeoPixel")
@@
  (footprint "RevK:C_0402"
   (layer "F.Cu")
-  (at 113.250000 85.600000 0)
+  (at 113.250000  109.250000)
   (property "Sheetfile" "5x7.kicad_sch")
   (property "Sheetname" "")
@@
  (footprint "RevK:SMD1010"
   (layer "F.Cu")
-  (at 109.250000 92.750000 135)
+  (at 109.250000  103.250000)
   (descr "https://cdn-shop.adafruit.com/datasheets/WS2812B.pdf")
   (tags "LED RGB NeoPixel")
@@
  (footprint "RevK:SMD1010"
   (layer "F.Cu")
-  (at 103.250000 90.750000 135)
+  (at 103.250000  105.250000)
   (descr "https://cdn-shop.adafruit.com/datasheets/WS2812B.pdf")
   (tags "LED RGB NeoPixel")
@@
  (footprint "RevK:C_0402"
   (layer "F.Cu")
-  (at 105.250000 85.600000 0)
+  (at 105.250000  105.250000)
   (property "Sheetfile" "5x7.kicad_sch")
   (property "Sheetname" "")
@@
  (footprint "RevK:SMD1010"
   (layer "F.Cu")
-  (at 105.250000 90.750000 135)
+  (at 105.250000  107.250000)
   (descr "https://cdn-shop.adafruit.com/datasheets/WS2812B.pdf")
   (tags "LED RGB NeoPixel")
@@
  (footprint "RevK:SMD1010"
   (layer "F.Cu")
-  (at 107.250000 92.750000 135)
+  (at 107.250000  105.250000)
   (descr "https://cdn-shop.adafruit.com/datasheets/WS2812B.pdf")
   (tags "LED RGB NeoPixel")
@@
  (footprint "RevK:SMD1010"
   (layer "F.Cu")
-  (at 105.250000 94.750000 135)
+  (at 105.250000  115.250000)
   (descr "https://cdn-shop.adafruit.com/datasheets/WS2812B.pdf")
   (tags "LED RGB NeoPixel")
@@
  (footprint "RevK:C_0402"
   (layer "F.Cu")
-  (at 115.250000 85.600000 0)
+  (at 115.250000  109.250000)
   (property "Sheetfile" "5x7.kicad_sch")
   (property "Sheetname" "")
@@
  (footprint "RevK:SMD1010"
   (layer "F.Cu")
-  (at 109.250000 96.750000 135)
+  (at 109.250000  111.250000)
   (descr "https://cdn-shop.adafruit.com/datasheets/WS2812B.pdf")
   (tags "LED RGB NeoPixel")
@@
  (footprint "RevK:C_0402"
   (layer "F.Cu")
-  (at 111.250000 99.900000 0)
+  (at 111.250000  107.250000)
   (property "Sheetfile" "5x7.kicad_sch")
   (property "Sheetname" "")
@@
  (footprint "RevK:SMD1010"
   (layer "F.Cu")
-  (at 107.250000 90.750000 135)
+  (at 107.250000  107.250000)
   (descr "https://cdn-shop.adafruit.com/datasheets/WS2812B.pdf")
   (tags "LED RGB NeoPixel")
@@
  (footprint "RevK:SMD1010"
   (layer "F.Cu")
-  (at 107.250000 94.750000 135)
+  (at 107.250000  105.250000)
   (descr "https://cdn-shop.adafruit.com/datasheets/WS2812B.pdf")
   (tags "LED RGB NeoPixel")
@@
  (footprint "RevK:SMD1010"
   (layer "F.Cu")
-  (at 105.250000 88.750000 135)
+  (at 105.250000  109.250000)
   (descr "https://cdn-shop.adafruit.com/datasheets/WS2812B.pdf")
   (tags "LED RGB NeoPixel")
@@
  (footprint "RevK:SMD1010"
   (layer "F.Cu")
-  (at 109.250000 94.750000 135)
+  (at 109.250000  105.250000)
   (descr "https://cdn-shop.adafruit.com/datasheets/WS2812B.pdf")
   (tags "LED RGB NeoPixel")
@@
  (footprint "RevK:SMD1010"
   (layer "F.Cu")
-  (at 105.250000 96.750000 135)
+  (at 105.250000  103.250000)
   (descr "https://cdn-shop.adafruit.com/datasheets/WS2812B.pdf")
   (tags "LED RGB NeoPixel")
@@
  (footprint "RevK:SMD1010"
   (layer "F.Cu")
-  (at 103.250000 86.750000 135)
+  (at 103.250000  105.250000)
   (descr "https://cdn-shop.adafruit.com/datasheets/WS2812B.pdf")
   (tags "LED RGB NeoPixel")
@@
  (footprint "RevK:SMD1010"
   (layer "F.Cu")
-  (at 105.250000 98.750000 135)
+  (at 105.250000  103.250000)
   (descr "https://cdn-shop.adafruit.com/datasheets/WS2812B.pdf")
   (tags "LED RGB NeoPixel")
@@
  (footprint "RevK:C_0402"
   (layer "F.Cu")
-  (at 103.250000 85.600000 0)
+  (at 103.250000  103.250000)
   (property "Sheetfile" "5x7.kicad_sch")
   (property "Sheetname" "")
@@
  (footprint "RevK:C_0402"
   (layer "F.Cu")
-  (at 103.250000 99.900000 0)
+  (at 103.250000  113.250000)
   (property "Sheetfile" "5x7.kicad_sch")
   (property "Sheetname" "")
@@
  (footprint "RevK:C_0402"
   (layer "F.Cu")
-  (at 113.250000 99.900000 0)
+  (at 113.250000  103.250000)
   (property "Sheetfile" "5x7.kicad_sch")
   (property "Sheetname" "")
@@
  (footprint "RevK:SMD1010"
   (layer "F.Cu")
-  (at 103.250000 96.750000 135)
+  (at 103.250000  109.250000)
   (descr "https://cdn-shop.adafruit.com/datasheets/WS2812B.pdf")
   (tags "LED RGB NeoPixel")
@@
  (footprint "RevK:C_0402"
   (layer "F.Cu")
-  (at 109.250000 85.600000 0)
+  (at 109.250000  107.250000)
   (property "Sheetfile" "5x7.kicad_sch")
   (property "Sheetname" "")
@@
  (footprint "RevK:SMD1010"
   (layer "F.Cu")
-  (at 107.250000 96.750000 135)
+  (at 107.250000  115.250000)
   (descr "https://cdn-shop.adafruit.com/datasheets/WS2812B.pdf")
   (tags "LED RGB NeoPixel")
@@
  (footprint "RevK:C_0402"
   (layer "F.Cu")
-  (at 115.250000 99.900000 0)
+  (at 115.250000  109.250000)
   (property "Sheetfile" "5x7.kicad_sch")
   (property "Sheetname" "")
@@
  (footprint "RevK:SMD1010"
   (layer "F.Cu")
-  (at 109.250000 86.750000 135)
+  (at 109.250000  109.250000)
   (descr "https://cdn-shop.adafruit.com/datasheets/WS2812B.pdf")
   (tags "LED RGB NeoPixel")
@@
  (footprint "RevK:SMD1010"
   (layer "F.Cu")
-  (at 109.250000 90.750000 135)
+  (at 109.250000  111.250000)
   (descr "https://cdn-shop.adafruit.com/datasheets/WS2812B.pdf")
   (tags "LED RGB NeoPixel")
@@
  (footprint "RevK:SMD1010"
   (layer "F.Cu")
-  (at 111.250000 94.750000 135)
+  (at 111.250000  111.250000)
   (descr "https://cdn-shop.adafruit.com/datasheets/WS2812B.pdf")
   (tags "LED RGB NeoPixel")
@@
  (footprint "RevK:SMD1010"
   (layer "F.Cu")
-  (at 111.250000 86.750000 135)
+  (at 111.250000  111.250000)
   (descr "https://cdn-shop.adafruit.com/datasheets/WS2812B.pdf")
   (tags "LED RGB NeoPixel")
@@
  (footprint "RevK:C_0402"
   (layer "F.Cu")
-  (at 111.250000 85.600000 0)
+  (at 111.250000  103.250000)
   (property "Sheetfile" "5x7.kicad_sch")
   (property "Sheetname" "")
@@
  (footprint "RevK:SMD1010"
   (layer "F.Cu")
-  (at 103.250000 92.750000 135)
+  (at 103.250000  105.250000)
   (descr "https://cdn-shop.adafruit.com/datasheets/WS2812B.pdf")
   (tags "LED RGB NeoPixel")
@@
  (footprint "RevK:C_0402"
   (layer "F.Cu")
-  (at 105.250000 99.900000 0)
+  (at 105.250000  109.250000)
   (property "Sheetfile" "5x7.kicad_sch")
   (property "Sheetname" "")
@@
  (footprint "RevK:SMD1010"
   (layer "F.Cu")
-  (at 109.250000 88.750000 135)
+  (at 109.250000  105.250000)
   (descr "https://cdn-shop.adafruit.com/datasheets/WS2812B.pdf")
   (tags "LED RGB NeoPixel")
@@
  (footprint "RevK:SMD1010"
   (layer "F.Cu")
-  (at 105.250000 92.750000 135)
+  (at 105.250000  107.250000)
   (descr "https://cdn-shop.adafruit.com/datasheets/WS2812B.pdf")
   (tags "LED RGB NeoPixel")
@@
  (footprint "RevK:C_0402"
   (layer "F.Cu")
-  (at 107.250000 99.900000 0)
+  (at 107.250000  111.250000)
   (property "Sheetfile" "5x7.kicad_sch")
   (property "Sheetname" "")
@@
  (footprint "RevK:SMD1010"
   (layer "F.Cu")
-  (at 111.250000 88.750000 135)
+  (at 111.250000  103.250000)
   (descr "https://cdn-shop.adafruit.com/datasheets/WS2812B.pdf")
   (tags "LED RGB NeoPixel")
@@
  (footprint "RevK:SMD1010"
   (layer "F.Cu")
-  (at 103.250000 94.750000 135)
+  (at 103.250000  111.250000)
   (descr "https://cdn-shop.adafruit.com/datasheets/WS2812B.pdf")
   (tags "LED RGB NeoPixel")
@@
  (footprint "RevK:SMD1010"
   (layer "F.Cu")
-  (at 111.250000 92.750000 135)
+  (at 111.250000  111.250000)
   (descr "https://cdn-shop.adafruit.com/datasheets/WS2812B.pdf")
   (tags "LED RGB NeoPixel")
@@
  (footprint "RevK:SMD1010"
   (layer "F.Cu")
-  (at 111.250000 96.750000 135)
+  (at 111.250000  103.250000)
   (descr "https://cdn-shop.adafruit.com/datasheets/WS2812B.pdf")
   (tags "LED RGB NeoPixel")
@@
  (footprint "RevK:SMD1010"
   (layer "F.Cu")
-  (at 103.250000 88.750000 135)
+  (at 103.250000  109.250000)
   (descr "https://cdn-shop.adafruit.com/datasheets/WS2812B.pdf")
   (tags "LED RGB NeoPixel")
@@
  (footprint "RevK:SMD1010"
   (layer "F.Cu")
-  (at 109.250000 98.750000 135)
+  (at 109.250000  107.250000)
   (descr "https://cdn-shop.adafruit.com/datasheets/WS2812B.pdf")
   (tags "LED RGB NeoPixel")
@@
  (footprint "RevK:C_0402"
   (layer "F.Cu")
-  (at 107.250000 85.600000 0)
+  (at 107.250000  111.250000)
   (property "Sheetfile" "5x7.kicad_sch")
   (property "Sheetname" "")
@@
  (footprint "RevK:SMD1010"
   (layer "F.Cu")
-  (at 111.250000 98.750000 135)
+  (at 111.250000  105.250000)
   (descr "https://cdn-shop.adafruit.com/datasheets/WS2812B.pdf")
   (tags "LED RGB NeoPixel")
@@
  (footprint "RevK:SMD1010"
   (layer "F.Cu")
-  (at 105.250000 86.750000 135)
+  (at 105.250000  111.250000)
   (descr "https://cdn-shop.adafruit.com/datasheets/WS2812B.pdf")
   (tags "LED RGB NeoPixel")
@@
  (footprint "RevK:SMD1010"
   (layer "F.Cu")
-  (at 111.250000 90.750000 135)
+  (at 111.250000  103.250000)
   (descr "https://cdn-shop.adafruit.com/datasheets/WS2812B.pdf")
   (tags "LED RGB NeoPixel")
@@
  (footprint "RevK:SMD1010"
   (layer "F.Cu")
-  (at 103.250000 98.750000 135)
+  (at 103.250000  109.250000)
   (descr "https://cdn-shop.adafruit.com/datasheets/WS2812B.pdf")
   (tags "LED RGB NeoPixel")
@@
  (footprint "RevK:C_0402"
   (layer "F.Cu")
-  (at 109.250000 99.900000 0)
+  (at 109.250000  107.250000)
   (property "Sheetfile" "5x7.kicad_sch")
   (property "Sheetname" "")
@@
  (footprint "RevK:SMD1010"
   (layer "F.Cu")
-  (at 107.250000 88.750000 135)
+  (at 107.250000  )
   (descr "https://cdn-shop.adafruit.com/datasheets/WS2812B.pdf")
   (tags "LED RGB NeoPixel")

Commit message: Indent
Parts:
- moved D16 151.7 mm to (107.2, 107.2), turned to 135 degrees
- moved C12 15.2 mm to (113.2, 118.4)
- moved D14 14.0 mm to (105.2, 117.2), turned to 135 degrees
- moved D13 12.0 mm to (105.2, 115.2), turned to 135 degrees
- moved D34 12.0 mm to (111.2, 115.2), turned to 135 degrees
- moved D35 12.0 mm to (111.2, 117.2), turned to 135 degrees
- moved C10 11.2 mm to (111.2, 118.4)
- moved C8 11.2 mm to (109.2, 118.4)
- moved D28 10.0 mm to (109.2, 117.2), turned to 135 degrees
- moved C14 9.15 mm to (115.2, 118.4)
- moved C4 9.15 mm to (105.2, 118.4)
- moved D19 8.00 mm to (107.2, 113.2), turned to 135 degrees
- moved D25 8.00 mm to (109.2, 111.2), turned to 135 degrees
- moved D26 8.00 mm to (109.2, 113.2), turned to 135 degrees
- moved D7 8.00 mm to (103.2, 117.2), turned to 135 degrees
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Changed lines of the file:
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@@
  (footprint "RevK:SMD1010"
   (layer "F.Cu")
-  (at 107.250000  107.250000)
+  (at 107.250000 105.250000 135)
   (descr "https://cdn-shop.adafruit.com/datasheets/WS2812B.pdf")
   (tags "LED RGB NeoPixel")
@@
  (footprint "RevK:SMD1010"
   (layer "F.Cu")
-  (at 107.250000  113.250000)
+  (at 107.250000 117.250000 135)
   (descr "https://cdn-shop.adafruit.com/datasheets/WS2812B.pdf")
   (tags "LED RGB NeoPixel")
@@
  (footprint "RevK:C_0402"
   (layer "F.Cu")
-  (at 113.250000  109.250000)
+  (at 113.250000 104.100000 0)
   (property "Sheetfile" "5x7.kicad_sch")
   (property "Sheetname" "")
@@
  (footprint "RevK:SMD1010"
   (layer "F.Cu")
-  (at 109.250000  103.250000)
+  (at 109.250000 111.250000 135)
   (descr "https://cdn-shop.adafruit.com/datasheets/WS2812B.pdf")
   (tags "LED RGB NeoPixel")
@@
  (footprint "RevK:SMD1010"
   (layer "F.Cu")
-  (at 103.250000  105.250000)
+  (at 103.250000 109.250000 135)
   (descr "https://cdn-shop.adafruit.com/datasheets/WS2812B.pdf")
   (tags "LED RGB NeoPixel")
@@
  (footprint "RevK:C_0402"
   (layer "F.Cu")
-  (at 105.250000  105.250000)
+  (at 105.250000 104.100000 0)
   (property "Sheetfile" "5x7.kicad_sch")
   (property "Sheetname" "")
@@
  (footprint "RevK:SMD1010"
   (layer "F.Cu")
-  (at 105.250000  107.250000)
+  (at 105.250000 109.250000 135)
   (descr "https://cdn-shop.adafruit.com/datasheets/WS2812B.pdf")
   (tags "LED RGB NeoPixel")
@@
  (footprint "RevK:SMD1010"
   (layer "F.Cu")
-  (at 107.250000  105.250000)
+  (at 107.250000 111.250000 135)
   (descr "https://cdn-shop.adafruit.com/datasheets/WS2812B.pdf")
   (tags "LED RGB NeoPixel")
@@
  (footprint "RevK:SMD1010"
   (layer "F.Cu")
-  (at 105.250000  115.250000)
+  (at 105.250000 113.250000 135)
   (descr "https://cdn-shop.adafruit.com/datasheets/WS2812B.pdf")
   (tags "LED RGB NeoPixel")
@@
  (footprint "RevK:C_0402"
   (layer "F.Cu")
-  (at 115.250000  109.250000)
+  (at 115.250000 104.100000 0)
   (property "Sheetfile" "5x7.kicad_sch")
   (property "Sheetname" "")
@@
  (footprint "RevK:SMD1010"
   (layer "F.Cu")
-  (at 109.250000  111.250000)
+  (at 109.250000 115.250000 135)
   (descr "https://cdn-shop.adafruit.com/datasheets/WS2812B.pdf")
   (tags "LED RGB NeoPixel")
@@
  (footprint "RevK:C_0402"
   (layer "F.Cu")
-  (at 111.250000  107.250000)
+  (at 111.250000 118.400000 0)
   (property "Sheetfile" "5x7.kicad_sch")
   (property "Sheetname" "")
@@
  (footprint "RevK:SMD1010"
   (layer "F.Cu")
-  (at 107.250000  107.250000)
+  (at 107.250000 109.250000 135)
   (descr "https://cdn-shop.adafruit.com/datasheets/WS2812B.pdf")
   (tags "LED RGB NeoPixel")
@@
  (footprint "RevK:SMD1010"
   (layer "F.Cu")
-  (at 107.250000  105.250000)
+  (at 107.250000 113.250000 135)
   (descr "https://cdn-shop.adafruit.com/datasheets/WS2812B.pdf")
   (tags "LED RGB NeoPixel")
@@
  (footprint "RevK:SMD1010"
   (layer "F.Cu")
-  (at 105.250000  109.250000)
+  (at 105.250000 107.250000 135)
   (descr "https://cdn-shop.adafruit.com/datasheets/WS2812B.pdf")
   (tags "LED RGB NeoPixel")
@@
  (footprint "RevK:SMD1010"
   (layer "F.Cu")
-  (at 109.250000  105.250000)
+  (at 109.250000 113.250000 135)
   (descr "https://cdn-shop.adafruit.com/datasheets/WS2812B.pdf")
   (tags "LED RGB NeoPixel")
@@
  (footprint "RevK:SMD1010"
   (layer "F.Cu")
-  (at 105.250000  103.250000)
+  (at 105.250000 115.250000 135)
   (descr "https://cdn-shop.adafruit.com/datasheets/WS2812B.pdf")
   (tags "LED RGB NeoPixel")
@@
  (footprint "RevK:SMD1010"
   (layer "F.Cu")
-  (at 103.250000  105.250000)
+  (at 103.250000 105.250000 135)
   (descr "https://cdn-shop.adafruit.com/datasheets/WS2812B.pdf")
   (tags "LED RGB NeoPixel")
@@
  (footprint "RevK:SMD1010"
   (layer "F.Cu")
-  (at 105.250000  103.250000)
+  (at 105.250000 117.250000 135)
   (descr "https://cdn-shop.adafruit.com/datasheets/WS2812B.pdf")
   (tags "LED RGB NeoPixel")
@@
  (footprint "RevK:C_0402"
   (layer "F.Cu")
-  (at 103.250000  103.250000)
+  (at 103.250000 104.100000 0)
   (property "Sheetfile" "5x7.kicad_sch")
   (property "Sheetname" "")
@@
  (footprint "RevK:C_0402"
   (layer "F.Cu")
-  (at 103.250000  113.250000)
+  (at 103.250000 118.400000 0)
   (property "Sheetfile" "5x7.kicad_sch")
   (property "Sheetname" "")
@@
  (footprint "RevK:C_0402"
   (layer "F.Cu")
-  (at 113.250000  103.250000)
+  (at 113.250000 118.400000 0)
   (property "Sheetfile" "5x7.kicad_sch")
   (property "Sheetname" "")
@@
  (footprint "RevK:SMD1010"
   (layer "F.Cu")
-  (at 103.250000  109.250000)
+  (at 103.250000 115.250000 135)
   (descr "https://cdn-shop.adafruit.com/datasheets/WS2812B.pdf")
   (tags "LED RGB NeoPixel")
@@
  (footprint "RevK:C_0402"
   (layer "F.Cu")
-  (at 109.250000  107.250000)
+  (at 109.250000 104.100000 0)
   (property "Sheetfile" "5x7.kicad_sch")
   (property "Sheetname" "")
@@
  (footprint "RevK:SMD1010"
   (layer "F.Cu")
-  (at 107.250000  115.250000)
+  (at 107.250000 115.250000 135)
   (descr "https://cdn-shop.adafruit.com/datasheets/WS2812B.pdf")
   (tags "LED RGB NeoPixel")
@@
  (footprint "RevK:C_0402"
   (layer "F.Cu")
-  (at 115.250000  109.250000)
+  (at 115.250000 118.400000 0)
   (property "Sheetfile" "5x7.kicad_sch")
   (property "Sheetname" "")
@@
  (footprint "RevK:SMD1010"
   (layer "F.Cu")
-  (at 109.250000  109.250000)
+  (at 109.250000 105.250000 135)
   (descr "https://cdn-shop.adafruit.com/datasheets/WS2812B.pdf")
   (tags "LED RGB NeoPixel")
@@
  (footprint "RevK:SMD1010"
   (layer "F.Cu")
-  (at 109.250000  111.250000)
+  (at 109.250000 109.250000 135)
   (descr "https://cdn-shop.adafruit.com/datasheets/WS2812B.pdf")
   (tags "LED RGB NeoPixel")
@@
  (footprint "RevK:SMD1010"
   (layer "F.Cu")
-  (at 111.250000  111.250000)
+  (at 111.250000 113.250000 135)
   (descr "https://cdn-shop.adafruit.com/datasheets/WS2812B.pdf")
   (tags "LED RGB NeoPixel")
@@
  (footprint "RevK:SMD1010"
   (layer "F.Cu")
-  (at 111.250000  111.250000)
+  (at 111.250000 105.250000 135)
   (descr "https://cdn-shop.adafruit.com/datasheets/WS2812B.pdf")
   (tags "LED RGB NeoPixel")
@@
  (footprint "RevK:C_0402"
   (layer "F.Cu")
-  (at 111.250000  103.250000)
+  (at 111.250000 104.100000 0)
   (property "Sheetfile" "5x7.kicad_sch")
   (property "Sheetname" "")
@@
  (footprint "RevK:SMD1010"
   (layer "F.Cu")
-  (at 103.250000  105.250000)
+  (at 103.250000 111.250000 135)
   (descr "https://cdn-shop.adafruit.com/datasheets/WS2812B.pdf")
   (tags "LED RGB NeoPixel")
@@
  (footprint "RevK:C_0402"
   (layer "F.Cu")
-  (at 105.250000  109.250000)
+  (at 105.250000 118.400000 0)
   (property "Sheetfile" "5x7.kicad_sch")
   (property "Sheetname" "")
@@
  (footprint "RevK:SMD1010"
   (layer "F.Cu")
-  (at 109.250000  105.250000)
+  (at 109.250000 107.250000 135)
   (descr "https://cdn-shop.adafruit.com/datasheets/WS2812B.pdf")
   (tags "LED RGB NeoPixel")
@@
  (footprint "RevK:SMD1010"
   (layer "F.Cu")
-  (at 105.250000  107.250000)
+  (at 105.250000 111.250000 135)
   (descr "https://cdn-shop.adafruit.com/datasheets/WS2812B.pdf")
   (tags "LED RGB NeoPixel")
@@
  (footprint "RevK:C_0402"
   (layer "F.Cu")
-  (at 107.250000  111.250000)
+  (at 107.250000 118.400000 0)
   (property "Sheetfile" "5x7.kicad_sch")
   (property "Sheetname" "")
@@
  (footprint "RevK:SMD1010"
   (layer "F.Cu")
-  (at 111.250000  103.250000)
+  (at 111.250000 107.250000 135)
   (descr "https://cdn-shop.adafruit.com/datasheets/WS2812B.pdf")
   (tags "LED RGB NeoPixel")
@@
  (footprint "RevK:SMD1010"
   (layer "F.Cu")
-  (at 103.250000  111.250000)
+  (at 103.250000 113.250000 135)
   (descr "https://cdn-shop.adafruit.com/datasheets/WS2812B.pdf")
   (tags "LED RGB NeoPixel")
@@
  (footprint "RevK:SMD1010"
   (layer "F.Cu")
-  (at 111.250000  111.250000)
+  (at 111.250000 111.250000 135)
   (descr "https://cdn-shop.adafruit.com/datasheets/WS2812B.pdf")
   (tags "LED RGB NeoPixel")
@@
  (footprint "RevK:SMD1010"
   (layer "F.Cu")
-  (at 111.250000  103.250000)
+  (at 111.250000 115.250000 135)
   (descr "https://cdn-shop.adafruit.com/datasheets/WS2812B.pdf")
   (tags "LED RGB NeoPixel")
@@
  (footprint "RevK:SMD1010"
   (layer "F.Cu")
-  (at 103.250000  109.250000)
+  (at 103.250000 107.250000 135)
   (descr "https://cdn-shop.adafruit.com/datasheets/WS2812B.pdf")
   (tags "LED RGB NeoPixel")
@@
  (footprint "RevK:SMD1010"
   (layer "F.Cu")
-  (at 109.250000  107.250000)
+  (at 109.250000 117.250000 135)
   (descr "https://cdn-shop.adafruit.com/datasheets/WS2812B.pdf")
   (tags "LED RGB NeoPixel")
@@
  (footprint "RevK:C_0402"
   (layer "F.Cu")
-  (at 107.250000  111.250000)
+  (at 107.250000 104.100000 0)
   (property "Sheetfile" "5x7.kicad_sch")
   (property "Sheetname" "")
@@
  (footprint "RevK:SMD1010"
   (layer "F.Cu")
-  (at 111.250000  105.250000)
+  (at 111.250000 117.250000 135)
   (descr "https://cdn-shop.adafruit.com/datasheets/WS2812B.pdf")
   (tags "LED RGB NeoPixel")
@@
  (footprint "RevK:SMD1010"
   (layer "F.Cu")
-  (at 105.250000  111.250000)
+  (at 105.250000 105.250000 135)
   (descr "https://cdn-shop.adafruit.com/datasheets/WS2812B.pdf")
   (tags "LED RGB NeoPixel")
@@
  (footprint "RevK:SMD1010"
   (layer "F.Cu")
-  (at 111.250000  103.250000)
+  (at 111.250000 109.250000 135)
   (descr "https://cdn-shop.adafruit.com/datasheets/WS2812B.pdf")
   (tags "LED RGB NeoPixel")
@@
  (footprint "RevK:SMD1010"
   (layer "F.Cu")
-  (at 103.250000  109.250000)
+  (at 103.250000 117.250000 135)
   (descr "https://cdn-shop.adafruit.com/datasheets/WS2812B.pdf")
   (tags "LED RGB NeoPixel")
@@
  (footprint "RevK:C_0402"
   (layer "F.Cu")
-  (at 109.250000  107.250000)
+  (at 109.250000 118.400000 0)
   (property "Sheetfile" "5x7.kicad_sch")
   (property "Sheetname" "")
@@
  (footprint "RevK:SMD1010"
   (layer "F.Cu")
-  (at 107.250000  )
+  (at 107.250000 107.250000 135)
   (descr "https://cdn-shop.adafruit.com/datasheets/WS2812B.pdf")
   (tags "LED RGB NeoPixel")
