File: PCB/Gate/Gate.kicad_pcb (KiCad board)
At the start: 2 copper layers, 398.5 x 198.3 mm, 200 parts, among them J1 Shelly, J2 USB-C, P1 TestPoint, P10 TestPoint, P11 TestPoint, P12 TestPoint, P13 TestPoint, P2 TestPoint, P3 TestPoint, P4 TestPoint, P5 TestPoint, P6 TestPoint, P7 TestPoint, P8 TestPoint, P9 TestPoint, T1 TestPoint, T10 TestPoint, T11 TestPoint, T12 TestPoint, T13 TestPoint, T2 TestPoint, T3 TestPoint, T4 TestPoint, T5 TestPoint, T6 TestPoint, T7 TestPoint, T8 TestPoint, T9 TestPoint, U1 QR, U2 ESP32-PICO-MINI-02, U3 LMR16006XDDCR

Commit message: Start on ring
Parts:
- removed H1, H10, H11, H12, H13, H14, H15, H16, H17, H18, H19, H2, H20, H21, H22, H23, H24, H25, H26, H27, H28, H29, H3, H30, H31, H32, H33, H34, H35, H36, H37, H38, H39, H4, H5, H6, H7, H8, H9: -, RevK:LEDHOLE
- removed J1: Shelly, RevK:Shelly
- removed J2: USB-C, RevK:USC16-TR
- removed L1: 6.8uH, RevK:L_4x4_
- removed P1, P10, P11, P12, P13, P2, P3, P4, P5, P6, P7, P8, P9: TestPoint, RevK:PAD
- removed R1: 10k, RevK:R_0603
- removed R2: 300R, RevK:R_0603
- removed R3: 100k 1%, RevK:R_0603
- removed R4: 30k 1%, RevK:R_0603
- removed R5, R6: 5K1, RevK:R_0603
- removed T1, T10, T11, T12, T13, T2, T3, T4, T5, T6, T7, T8, T9: TestPoint, RevK:PAD-LINK
- removed U2: ESP32-PICO-MINI-02, RevK:ESP32-PICO-MINI-02
- removed U3: LMR16006XDDCR, RevK:SOT-23-Thin-6-Reg
- added C100: 330nF, RevK:C_0402, F.Cu at (208.9, 79.8)
- added C101: 330nF, RevK:C_0402, F.Cu at (209.4, 80.6)
- added C102: 330nF, RevK:C_0402, F.Cu at (210.0, 81.5)
- added C103: 330nF, RevK:C_0402, F.Cu at (210.5, 82.3)
- added C104: 330nF, RevK:C_0402, F.Cu at (211.0, 83.2)
- added C105: 330nF, RevK:C_0402, F.Cu at (211.5, 84.1)
- added C106: 330nF, RevK:C_0402, F.Cu at (212.0, 84.9)
- added C107: 330nF, RevK:C_0402, F.Cu at (212.5, 85.8)
- added C108: 330nF, RevK:C_0402, F.Cu at (213.0, 86.7)
- added C109: 330nF, RevK:C_0402, F.Cu at (213.4, 87.6)
- added C110: 330nF, RevK:C_0402, F.Cu at (213.9, 88.4)
- added C111: 330nF, RevK:C_0402, F.Cu at (214.4, 89.3)
- added C112: 330nF, RevK:C_0402, F.Cu at (214.8, 90.2)
- added C113: 330nF, RevK:C_0402, F.Cu at (215.2, 91.1)
- added C114: 330nF, RevK:C_0402, F.Cu at (215.7, 92.0)
- added C115: 330nF, RevK:C_0402, F.Cu at (216.1, 93.0)
- added C116: 330nF, RevK:C_0402, F.Cu at (216.5, 93.9)
- added C117: 330nF, RevK:C_0402, F.Cu at (216.9, 94.8)
- added C83: 330nF, RevK:C_0402, F.Cu at (198.5, 66.4)
- added C84: 330nF, RevK:C_0402, F.Cu at (199.1, 67.1)
- added C85: 330nF, RevK:C_0402, F.Cu at (199.8, 67.9)
- added C86: 330nF, RevK:C_0402, F.Cu at (200.5, 68.6)
- added C87: 330nF, RevK:C_0402, F.Cu at (201.1, 69.4)
- added C88: 330nF, RevK:C_0402, F.Cu at (201.8, 70.1)
- added C89: 330nF, RevK:C_0402, F.Cu at (202.4, 70.9)
- added C90: 330nF, RevK:C_0402, F.Cu at (203.0, 71.7)
- added C91: 330nF, RevK:C_0402, F.Cu at (203.7, 72.5)
- added C92: 330nF, RevK:C_0402, F.Cu at (204.3, 73.3)
- added C93: 330nF, RevK:C_0402, F.Cu at (204.9, 74.1)
- added C94: 330nF, RevK:C_0402, F.Cu at (205.5, 74.9)
- added C95: 330nF, RevK:C_0402, F.Cu at (206.1, 75.7)
- added C96: 330nF, RevK:C_0402, F.Cu at (206.6, 76.5)
- added C97: 330nF, RevK:C_0402, F.Cu at (207.2, 77.3)
- added C98: 330nF, RevK:C_0402, F.Cu at (207.8, 78.1)
- added C99: 330nF, RevK:C_0402, F.Cu at (208.3, 79.0)
- added D100: XL-1010RGBC-WS2812B, RevK:SMD1010, F.Cu at (208.6, 79.4)
- added D101: XL-1010RGBC-WS2812B, RevK:SMD1010, F.Cu at (209.2, 80.2)
- added D102: XL-1010RGBC-WS2812B, RevK:SMD1010, F.Cu at (209.7, 81.1)
- added D103: XL-1010RGBC-WS2812B, RevK:SMD1010, F.Cu at (210.2, 81.9)
- added D104: XL-1010RGBC-WS2812B, RevK:SMD1010, F.Cu at (210.7, 82.8)
- added D105: XL-1010RGBC-WS2812B, RevK:SMD1010, F.Cu at (211.2, 83.6)
- added D106: XL-1010RGBC-WS2812B, RevK:SMD1010, F.Cu at (211.7, 84.5)
- added D107: XL-1010RGBC-WS2812B, RevK:SMD1010, F.Cu at (212.2, 85.4)
- added D108: XL-1010RGBC-WS2812B, RevK:SMD1010, F.Cu at (212.7, 86.2)
- added D109: XL-1010RGBC-WS2812B, RevK:SMD1010, F.Cu at (213.2, 87.1)
- added D110: XL-1010RGBC-WS2812B, RevK:SMD1010, F.Cu at (213.7, 88.0)
- added D111: XL-1010RGBC-WS2812B, RevK:SMD1010, F.Cu at (214.1, 88.9)
- added D112: XL-1010RGBC-WS2812B, RevK:SMD1010, F.Cu at (214.6, 89.8)
- added D113: XL-1010RGBC-WS2812B, RevK:SMD1010, F.Cu at (215.0, 90.7)
- added D114: XL-1010RGBC-WS2812B, RevK:SMD1010, F.Cu at (215.4, 91.6)
- added D115: XL-1010RGBC-WS2812B, RevK:SMD1010, F.Cu at (215.9, 92.5)
- added D116: XL-1010RGBC-WS2812B, RevK:SMD1010, F.Cu at (216.3, 93.4)
- added D117: XL-1010RGBC-WS2812B, RevK:SMD1010, F.Cu at (216.7, 94.3)
- added D41: XL-1010RGBC-WS2812B, RevK:SMD1010, F.Cu at (163.9, 42.1)
- added D42: XL-1010RGBC-WS2812B, RevK:SMD1010, F.Cu at (164.9, 42.5)
- added D43: XL-1010RGBC-WS2812B, RevK:SMD1010, F.Cu at (165.8, 42.9)
- added D44: XL-1010RGBC-WS2812B, RevK:SMD1010, F.Cu at (166.7, 43.3)
- added D45: XL-1010RGBC-WS2812B, RevK:SMD1010, F.Cu at (167.6, 43.7)
- added D46: XL-1010RGBC-WS2812B, RevK:SMD1010, F.Cu at (168.5, 44.2)
- added D47: XL-1010RGBC-WS2812B, RevK:SMD1010, F.Cu at (169.4, 44.6)
- added D48: XL-1010RGBC-WS2812B, RevK:SMD1010, F.Cu at (170.3, 45.1)
- added D49: XL-1010RGBC-WS2812B, RevK:SMD1010, F.Cu at (171.2, 45.5)
- added D50: XL-1010RGBC-WS2812B, RevK:SMD1010, F.Cu at (172.1, 46.0)
- added D51: XL-1010RGBC-WS2812B, RevK:SMD1010, F.Cu at (172.9, 46.5)
- added D52: XL-1010RGBC-WS2812B, RevK:SMD1010, F.Cu at (173.8, 46.9)
- added D53: XL-1010RGBC-WS2812B, RevK:SMD1010, F.Cu at (174.7, 47.4)
- added D54: XL-1010RGBC-WS2812B, RevK:SMD1010, F.Cu at (175.6, 47.9)
- added D55: XL-1010RGBC-WS2812B, RevK:SMD1010, F.Cu at (176.4, 48.4)
- added D56: XL-1010RGBC-WS2812B, RevK:SMD1010, F.Cu at (177.3, 49.0)
- added D57: XL-1010RGBC-WS2812B, RevK:SMD1010, F.Cu at (178.1, 49.5)
- added D58: XL-1010RGBC-WS2812B, RevK:SMD1010, F.Cu at (179.0, 50.0)
- added D59: XL-1010RGBC-WS2812B, RevK:SMD1010, F.Cu at (179.8, 50.6)
- added D60: XL-1010RGBC-WS2812B, RevK:SMD1010, F.Cu at (180.6, 51.1)
- added D61: XL-1010RGBC-WS2812B, RevK:SMD1010, F.Cu at (181.5, 51.7)
- added D62: XL-1010RGBC-WS2812B, RevK:SMD1010, F.Cu at (182.3, 52.3)
- added D63: XL-1010RGBC-WS2812B, RevK:SMD1010, F.Cu at (183.1, 52.8)
- added D64: XL-1010RGBC-WS2812B, RevK:SMD1010, F.Cu at (183.9, 53.4)
- added D65: XL-1010RGBC-WS2812B, RevK:SMD1010, F.Cu at (184.7, 54.0)
- added D66: XL-1010RGBC-WS2812B, RevK:SMD1010, F.Cu at (185.5, 54.6)
- added D67: XL-1010RGBC-WS2812B, RevK:SMD1010, F.Cu at (186.3, 55.2)
- added D68: XL-1010RGBC-WS2812B, RevK:SMD1010, F.Cu at (187.1, 55.8)
- added D69: XL-1010RGBC-WS2812B, RevK:SMD1010, F.Cu at (187.9, 56.5)
- added D70: XL-1010RGBC-WS2812B, RevK:SMD1010, F.Cu at (188.7, 57.1)
- added D71: XL-1010RGBC-WS2812B, RevK:SMD1010, F.Cu at (189.4, 57.7)
- added D72: XL-1010RGBC-WS2812B, RevK:SMD1010, F.Cu at (190.2, 58.4)
- added D73: XL-1010RGBC-WS2812B, RevK:SMD1010, F.Cu at (190.9, 59.0)
- added D74: XL-1010RGBC-WS2812B, RevK:SMD1010, F.Cu at (191.7, 59.7)
- added D75: XL-1010RGBC-WS2812B, RevK:SMD1010, F.Cu at (192.4, 60.4)
- added D76: XL-1010RGBC-WS2812B, RevK:SMD1010, F.Cu at (193.2, 61.1)
- added D77: XL-1010RGBC-WS2812B, RevK:SMD1010, F.Cu at (193.9, 61.7)
- added D78: XL-1010RGBC-WS2812B, RevK:SMD1010, F.Cu at (194.6, 62.4)
- added D79: XL-1010RGBC-WS2812B, RevK:SMD1010, F.Cu at (195.3, 63.1)
- added D80: XL-1010RGBC-WS2812B, RevK:SMD1010, F.Cu at (196.0, 63.8)
- added D81: XL-1010RGBC-WS2812B, RevK:SMD1010, F.Cu at (196.7, 64.6)
- added D82: XL-1010RGBC-WS2812B, RevK:SMD1010, F.Cu at (197.4, 65.3)
- added D83: XL-1010RGBC-WS2812B, RevK:SMD1010, F.Cu at (198.1, 66.0)
- added D84: XL-1010RGBC-WS2812B, RevK:SMD1010, F.Cu at (198.8, 66.7)
- added D85: XL-1010RGBC-WS2812B, RevK:SMD1010, F.Cu at (199.5, 67.5)
- added D86: XL-1010RGBC-WS2812B, RevK:SMD1010, F.Cu at (200.1, 68.2)
- added D87: XL-1010RGBC-WS2812B, RevK:SMD1010, F.Cu at (200.8, 69.0)
- added D88: XL-1010RGBC-WS2812B, RevK:SMD1010, F.Cu at (201.4, 69.8)
- added D89: XL-1010RGBC-WS2812B, RevK:SMD1010, F.Cu at (202.1, 70.5)
- added D90: XL-1010RGBC-WS2812B, RevK:SMD1010, F.Cu at (202.7, 71.3)
- added D91: XL-1010RGBC-WS2812B, RevK:SMD1010, F.Cu at (203.3, 72.1)
- added D92: XL-1010RGBC-WS2812B, RevK:SMD1010, F.Cu at (204.0, 72.9)
- added D93: XL-1010RGBC-WS2812B, RevK:SMD1010, F.Cu at (204.6, 73.7)
- added D94: XL-1010RGBC-WS2812B, RevK:SMD1010, F.Cu at (205.2, 74.5)
- added D95: XL-1010RGBC-WS2812B, RevK:SMD1010, F.Cu at (205.8, 75.3)
- added D96: XL-1010RGBC-WS2812B, RevK:SMD1010, F.Cu at (206.3, 76.1)
- added D97: XL-1010RGBC-WS2812B, RevK:SMD1010, F.Cu at (206.9, 76.9)
- added D98: XL-1010RGBC-WS2812B, RevK:SMD1010, F.Cu at (207.5, 77.7)
- added D99: XL-1010RGBC-WS2812B, RevK:SMD1010, F.Cu at (208.1, 78.5)
- C1, C10, C11, C12, C13, C14, C15, C16, C17, C18, C19, C2, C20, C21, C22, C23, C24, C25, C26, C27, C28, C29, C3, C30, C31, C32, C33, C34, C35, C36, C37, C38, C39, C4, C40, C41, C42, C43, C44, C45, C46, C47, C48, C49, C5, C50, C51, C52, C53, C54, C55, C56, C57, C58, C59, C6, C60, C61, C62, C63, C64, C65, C66, C67, C68, C69, C7, C70, C71, C72, C73, C74, C75, C76, C77, C78, C8, C9: value - -> 330nF; footprint RevK:C_0603 -> RevK:C_0402
- C79: value 10nF -> 330nF; footprint Capacitor_SMD:C_0603_1608Metric -> RevK:C_0402
- C80: value 100nF -> 330nF; footprint RevK:C_0603_ -> RevK:C_0402
- C81: value 2.2uF -> 330nF; footprint RevK:C_0805_ -> RevK:C_0402
- C82: value 10uF -> 330nF; footprint RevK:C_0805_ -> RevK:C_0402
- D1, D10, D11, D12, D13, D14, D15, D16, D17, D18, D19, D2, D20, D21, D22, D23, D24, D25, D26, D27, D28, D29, D3, D30, D31, D32, D33, D34, D35, D36, D37, D38, D39, D4, D5, D6, D7, D8, D9: value - -> XL-1010RGBC-WS2812B; footprint RevK:SMD2020 -> RevK:SMD1010
- D40: value Schottky -> XL-1010RGBC-WS2812B; footprint RevK:D_1206_ -> RevK:SMD1010
- moved C1 196.9 mm to (125.5, 34.2), turned to 90 degrees
- moved D33 196.1 mm to (156.5, 39.3), turned to -61.6242 degrees
- moved D1 195.9 mm to (125.0, 34.2), turned to -135 degrees
- moved D34 195.5 mm to (157.4, 39.6), turned to -59.3312 degrees
- moved C33 195.4 mm to (156.9, 39.4), turned to 163.376 degrees
- moved D32 195.4 mm to (155.5, 39.0), turned to -63.9172 degrees
- moved C34 195.1 mm to (157.9, 39.8), turned to 165.669 degrees
- moved C32 194.6 mm to (156.0, 39.1), turned to 161.083 degrees
- moved D35 193.8 mm to (158.3, 39.9), turned to -57.0382 degrees
- moved D31 193.6 mm to (154.5, 38.7), turned to -66.2102 degrees
- moved C35 193.5 mm to (158.8, 40.1), turned to 167.962 degrees
- moved C31 192.5 mm to (155.0, 38.8), turned to 158.79 degrees
- moved D36 190.8 mm to (159.3, 40.3), turned to -54.7452 degrees
- moved C36 190.7 mm to (159.8, 40.4), turned to 170.255 degrees
- moved D30 190.4 mm to (153.6, 38.4), turned to -68.5032 degrees
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Connections:
- C79 pad 1: GND -> VCC
- C79 pad 2: Net-(C79-Pad2) -> GND
Routing:
- net (no net): track 27.0 -> 0.00 mm
- net Net-(D31-Pad3): track 13.5 -> 0.00 mm
- net Net-(D14-Pad3): track 13.5 -> 0.00 mm
- net Net-(D2-Pad3): track 13.5 -> 0.00 mm
- net Net-(D26-Pad3): track 13.5 -> 0.00 mm
- net Net-(D21-Pad3): track 13.5 -> 0.00 mm
- net Net-(D16-Pad3): track 13.5 -> 0.00 mm
- net Net-(D17-Pad3): track 13.5 -> 0.00 mm
- net Net-(D7-Pad3): track 13.5 -> 0.00 mm
- net Net-(D29-Pad3): track 13.5 -> 0.00 mm
- net Net-(D10-Pad3): track 13.5 -> 0.00 mm
- net Net-(D37-Pad3): track 13.5 -> 0.00 mm
- net Net-(D24-Pad3): track 13.5 -> 0.00 mm
- net Net-(D15-Pad3): track 13.5 -> 0.00 mm
- net Net-(D34-Pad3): track 13.5 -> 0.00 mm
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- removed copper zone on F.Cu, net GND
- removed copper zone on B.Cu, net GND2
- removed copper zone on F.Cu, net GND2
- removed copper zone on F.Cu, net VCC
Other:
- board outline removed
- board text removed: "${DATE}"
- board text removed: "LED GPIO 22"

Commit message: Zone fill
Parts:
- moved C88 154.8 mm to (50.0, 100.7), turned to -179.231 degrees
- moved D88 154.8 mm to (50.0, 102.0), turned to -402.692 degrees
- moved D89 154.8 mm to (50.0, 99.3), turned to -405.769 degrees
- moved C87 154.8 mm to (50.1, 103.4), turned to -176.154 degrees
- moved C89 154.7 mm to (50.0, 98.0), turned to -182.308 degrees
- moved D87 154.7 mm to (50.2, 104.7), turned to -399.615 degrees
- moved D90 154.7 mm to (50.1, 96.6), turned to -408.846 degrees
- moved C86 154.7 mm to (50.4, 106.0), turned to -173.077 degrees
- moved C90 154.6 mm to (50.2, 95.3), turned to -185.385 degrees
- moved D86 154.6 mm to (50.5, 107.4), turned to -396.538 degrees
- moved D91 154.5 mm to (50.4, 94.0), turned to -411.923 degrees
- moved C85 154.5 mm to (50.8, 108.7), turned to -170 degrees
- moved C91 154.4 mm to (50.5, 92.6), turned to -188.462 degrees
- moved D85 154.4 mm to (51.0, 110.0), turned to -393.462 degrees
- moved D92 154.3 mm to (50.8, 91.3), turned to -415 degrees
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Routing:
- net (no net): track 0.00 -> 800.0 mm, vias 0 -> 2
- added copper zone on F.Cu, net GND
- added copper zone on F.Cu, net VCC
Other:
- board outline added: 124 x 124 mm

Commit message: Gate done
Parts:
- added C118: 330nF, RevK:C_0402, F.Cu at (104.8, 40.2)
- added C119: 330nF, RevK:C_0402, F.Cu at (114.4, 41.7)
- added C120: 330nF, RevK:C_0402, F.Cu at (123.5, 44.8)
- added C121: 330nF, RevK:C_0402, F.Cu at (132.1, 49.3)
- added C122: 330nF, RevK:C_0402, F.Cu at (139.8, 55.1)
- added C123: 330nF, RevK:C_0402, F.Cu at (146.5, 62.1)
- added C124: 330nF, RevK:C_0402, F.Cu at (152.0, 70.0)
- added C125: 330nF, RevK:C_0402, F.Cu at (156.1, 78.7)
- added C126: 330nF, RevK:C_0402, F.Cu at (158.8, 88.0)
- added C127: 330nF, RevK:C_0402, F.Cu at (160.0, 97.6)
- added C128: 330nF, RevK:C_0402, F.Cu at (159.6, 107.2)
- added C129: 330nF, RevK:C_0402, F.Cu at (157.6, 116.7)
- added C130: 330nF, RevK:C_0402, F.Cu at (154.2, 125.7)
- added C131: 330nF, RevK:C_0402, F.Cu at (149.4, 134.1)
- added C132: 330nF, RevK:C_0402, F.Cu at (143.3, 141.6)
- added C133: 330nF, RevK:C_0402, F.Cu at (136.0, 148.0)
- added C134: 330nF, RevK:C_0402, F.Cu at (127.9, 153.1)
- added C135: 330nF, RevK:C_0402, F.Cu at (119.0, 156.9)
- added C136: 330nF, RevK:C_0402, F.Cu at (109.6, 159.2)
- added C137: 330nF, RevK:C_0402, F.Cu at (100.0, 160.0)
- added C138: 330nF, RevK:C_0402, F.Cu at (90.4, 159.2)
- added C139: 330nF, RevK:C_0402, F.Cu at (81.0, 156.9)
- added C140: 330nF, RevK:C_0402, F.Cu at (72.1, 153.1)
- added C141: 330nF, RevK:C_0402, F.Cu at (64.0, 148.0)
- added C142: 330nF, RevK:C_0402, F.Cu at (56.7, 141.6)
- added C143: 330nF, RevK:C_0402, F.Cu at (50.6, 134.1)
- added C144: 330nF, RevK:C_0402, F.Cu at (45.8, 125.7)
- added C145: 330nF, RevK:C_0402, F.Cu at (42.4, 116.7)
- added C146: 330nF, RevK:C_0402, F.Cu at (40.4, 107.2)
- added C147: 330nF, RevK:C_0402, F.Cu at (40.0, 97.6)
- added C148: 330nF, RevK:C_0402, F.Cu at (41.2, 88.0)
- added C149: 330nF, RevK:C_0402, F.Cu at (43.9, 78.7)
- added C150: 330nF, RevK:C_0402, F.Cu at (48.0, 70.0)
- added C151: 330nF, RevK:C_0402, F.Cu at (53.5, 62.1)
- added C152: 330nF, RevK:C_0402, F.Cu at (60.2, 55.1)
- added C153: 330nF, RevK:C_0402, F.Cu at (67.9, 49.3)
- added C154: 330nF, RevK:C_0402, F.Cu at (76.5, 44.8)
- added C155: 330nF, RevK:C_0402, F.Cu at (85.6, 41.7)
- added C156: 330nF, RevK:C_0402, F.Cu at (95.2, 40.2)
- added C157: 330nF, RevK:C_0402, F.Cu at (100.0, 47.5)
- added C158: 330nF, RevK:C_0402, F.Cu at (118.0, 50.7)
- added C159: 330nF, RevK:C_0402, F.Cu at (133.7, 59.8)
- added C160: 330nF, RevK:C_0402, F.Cu at (145.5, 73.8)
- added C161: 330nF, RevK:C_0402, F.Cu at (151.7, 90.9)
- added C162: 330nF, RevK:C_0402, F.Cu at (151.7, 109.1)
- added C163: 330nF, RevK:C_0402, F.Cu at (145.5, 126.2)
- added C164: 330nF, RevK:C_0402, F.Cu at (133.7, 140.2)
- added C165: 330nF, RevK:C_0402, F.Cu at (118.0, 149.3)
- added C166: 330nF, RevK:C_0402, F.Cu at (100.0, 152.5)
- added C167: 330nF, RevK:C_0402, F.Cu at (82.0, 149.3)
- added C168: 330nF, RevK:C_0402, F.Cu at (66.3, 140.2)
- added C169: 330nF, RevK:C_0402, F.Cu at (54.5, 126.2)
- added C170: 330nF, RevK:C_0402, F.Cu at (48.3, 109.1)
- added C171: 330nF, RevK:C_0402, F.Cu at (48.3, 90.9)
- added C172: 330nF, RevK:C_0402, F.Cu at (54.5, 73.8)
- added C173: 330nF, RevK:C_0402, F.Cu at (66.3, 59.8)
- added C174: 330nF, RevK:C_0402, F.Cu at (82.0, 50.7)
- added C175: 330nF, RevK:C_0402, F.Cu at (100.0, 45.0)
- added C176: 330nF, RevK:C_0402, F.Cu at (118.8, 48.3)
- added C177: 330nF, RevK:C_0402, F.Cu at (135.4, 57.9)
- added C178: 330nF, RevK:C_0402, F.Cu at (147.6, 72.5)
- added C179: 330nF, RevK:C_0402, F.Cu at (154.2, 90.4)
- added C180: 330nF, RevK:C_0402, F.Cu at (154.2, 109.6)
- added C181: 330nF, RevK:C_0402, F.Cu at (147.6, 127.5)
- added C182: 330nF, RevK:C_0402, F.Cu at (135.4, 142.1)
- added C183: 330nF, RevK:C_0402, F.Cu at (118.8, 151.7)
- added C184: 330nF, RevK:C_0402, F.Cu at (100.0, 155.0)
- added C185: 330nF, RevK:C_0402, F.Cu at (81.2, 151.7)
- added C186: 330nF, RevK:C_0402, F.Cu at (64.6, 142.1)
- added C187: 330nF, RevK:C_0402, F.Cu at (52.4, 127.5)
- added C188: 330nF, RevK:C_0402, F.Cu at (45.8, 109.6)
- added C189: 330nF, RevK:C_0402, F.Cu at (45.8, 90.4)
- added C190: 330nF, RevK:C_0402, F.Cu at (52.4, 72.5)
- added C191: 330nF, RevK:C_0402, F.Cu at (64.6, 57.9)
- added C192: 330nF, RevK:C_0402, F.Cu at (81.2, 48.3)
- added C193: 330nF, RevK:C_0402, F.Cu at (100.0, 42.5)
- added C194: 330nF, RevK:C_0402, F.Cu at (119.7, 46.0)
- added C195: 330nF, RevK:C_0402, F.Cu at (137.0, 56.0)
- added C196: 330nF, RevK:C_0402, F.Cu at (149.8, 71.2)
- added C197: 330nF, RevK:C_0402, F.Cu at (156.6, 90.0)
- added C198: 330nF, RevK:C_0402, F.Cu at (156.6, 110.0)
- added C199: 330nF, RevK:C_0402, F.Cu at (149.8, 128.8)
- added C200: 330nF, RevK:C_0402, F.Cu at (137.0, 144.0)
- added C201: 330nF, RevK:C_0402, F.Cu at (119.7, 154.0)
- added C202: 330nF, RevK:C_0402, F.Cu at (100.0, 157.5)
- added C203: 330nF, RevK:C_0402, F.Cu at (80.3, 154.0)
- added C204: 330nF, RevK:C_0402, F.Cu at (63.0, 144.0)
- added C205: 330nF, RevK:C_0402, F.Cu at (50.2, 128.8)
- added C206: 330nF, RevK:C_0402, F.Cu at (43.4, 110.0)
- added C207: 330nF, RevK:C_0402, F.Cu at (43.4, 90.0)
- added C208: 330nF, RevK:C_0402, F.Cu at (50.2, 71.2)
- added C209: 330nF, RevK:C_0402, F.Cu at (63.0, 56.0)
- added C210: 330nF, RevK:C_0402, F.Cu at (80.3, 46.0)
- added D118: XL-1010RGBC-WS2812B, RevK:SMD1010, F.Cu at (100.0, 40.0)
- added D119: XL-1010RGBC-WS2812B, RevK:SMD1010, F.Cu at (109.6, 40.8)
- added D120: XL-1010RGBC-WS2812B, RevK:SMD1010, F.Cu at (119.0, 43.1)
- added D121: XL-1010RGBC-WS2812B, RevK:SMD1010, F.Cu at (127.9, 46.9)
- added D122: XL-1010RGBC-WS2812B, RevK:SMD1010, F.Cu at (136.0, 52.0)
- added D123: XL-1010RGBC-WS2812B, RevK:SMD1010, F.Cu at (143.3, 58.4)
- added D124: XL-1010RGBC-WS2812B, RevK:SMD1010, F.Cu at (149.4, 65.9)
- added D125: XL-1010RGBC-WS2812B, RevK:SMD1010, F.Cu at (154.2, 74.3)
- added D126: XL-1010RGBC-WS2812B, RevK:SMD1010, F.Cu at (157.6, 83.3)
- added D127: XL-1010RGBC-WS2812B, RevK:SMD1010, F.Cu at (159.6, 92.8)
- added D128: XL-1010RGBC-WS2812B, RevK:SMD1010, F.Cu at (160.0, 102.4)
- added D129: XL-1010RGBC-WS2812B, RevK:SMD1010, F.Cu at (158.8, 112.0)
- added D130: XL-1010RGBC-WS2812B, RevK:SMD1010, F.Cu at (156.1, 121.3)
- added D131: XL-1010RGBC-WS2812B, RevK:SMD1010, F.Cu at (152.0, 130.0)
- added D132: XL-1010RGBC-WS2812B, RevK:SMD1010, F.Cu at (146.5, 137.9)
- added D133: XL-1010RGBC-WS2812B, RevK:SMD1010, F.Cu at (139.8, 144.9)
- added D134: XL-1010RGBC-WS2812B, RevK:SMD1010, F.Cu at (132.1, 150.7)
- added D135: XL-1010RGBC-WS2812B, RevK:SMD1010, F.Cu at (123.5, 155.2)
- added D136: XL-1010RGBC-WS2812B, RevK:SMD1010, F.Cu at (114.4, 158.3)
- added D137: XL-1010RGBC-WS2812B, RevK:SMD1010, F.Cu at (104.8, 159.8)
- added D138: XL-1010RGBC-WS2812B, RevK:SMD1010, F.Cu at (95.2, 159.8)
- added D139: XL-1010RGBC-WS2812B, RevK:SMD1010, F.Cu at (85.6, 158.3)
- added D140: XL-1010RGBC-WS2812B, RevK:SMD1010, F.Cu at (76.5, 155.2)
- added D141: XL-1010RGBC-WS2812B, RevK:SMD1010, F.Cu at (67.9, 150.7)
- added D142: XL-1010RGBC-WS2812B, RevK:SMD1010, F.Cu at (60.2, 144.9)
- added D143: XL-1010RGBC-WS2812B, RevK:SMD1010, F.Cu at (53.5, 137.9)
- added D144: XL-1010RGBC-WS2812B, RevK:SMD1010, F.Cu at (48.0, 130.0)
- added D145: XL-1010RGBC-WS2812B, RevK:SMD1010, F.Cu at (43.9, 121.3)
- added D146: XL-1010RGBC-WS2812B, RevK:SMD1010, F.Cu at (41.2, 112.0)
- added D147: XL-1010RGBC-WS2812B, RevK:SMD1010, F.Cu at (40.0, 102.4)
- added D148: XL-1010RGBC-WS2812B, RevK:SMD1010, F.Cu at (40.4, 92.8)
- added D149: XL-1010RGBC-WS2812B, RevK:SMD1010, F.Cu at (42.4, 83.3)
- added D150: XL-1010RGBC-WS2812B, RevK:SMD1010, F.Cu at (45.8, 74.3)
- added D151: XL-1010RGBC-WS2812B, RevK:SMD1010, F.Cu at (50.6, 65.9)
- added D152: XL-1010RGBC-WS2812B, RevK:SMD1010, F.Cu at (56.7, 58.4)
- added D153: XL-1010RGBC-WS2812B, RevK:SMD1010, F.Cu at (64.0, 52.0)
- added D154: XL-1010RGBC-WS2812B, RevK:SMD1010, F.Cu at (72.1, 46.9)
- added D155: XL-1010RGBC-WS2812B, RevK:SMD1010, F.Cu at (81.0, 43.1)
- added D156: XL-1010RGBC-WS2812B, RevK:SMD1010, F.Cu at (90.4, 40.8)
- added D157: XL-1010RGBC-WS2812B, RevK:SMD1010, F.Cu at (96.0, 47.7)
- added D158: XL-1010RGBC-WS2812B, RevK:SMD1010, F.Cu at (104.0, 47.7)
- added D159: XL-1010RGBC-WS2812B, RevK:SMD1010, F.Cu at (130.6, 57.3)
- added D160: XL-1010RGBC-WS2812B, RevK:SMD1010, F.Cu at (136.7, 62.5)
- added D161: XL-1010RGBC-WS2812B, RevK:SMD1010, F.Cu at (150.9, 87.0)
- added D162: XL-1010RGBC-WS2812B, RevK:SMD1010, F.Cu at (152.2, 94.8)
- added D163: XL-1010RGBC-WS2812B, RevK:SMD1010, F.Cu at (147.3, 122.7)
- added D164: XL-1010RGBC-WS2812B, RevK:SMD1010, F.Cu at (143.3, 129.6)
- added D165: XL-1010RGBC-WS2812B, RevK:SMD1010, F.Cu at (121.7, 147.8)
- added D166: XL-1010RGBC-WS2812B, RevK:SMD1010, F.Cu at (114.1, 150.6)
- added D167: XL-1010RGBC-WS2812B, RevK:SMD1010, F.Cu at (85.9, 150.6)
- added D168: XL-1010RGBC-WS2812B, RevK:SMD1010, F.Cu at (78.3, 147.8)
- added D169: XL-1010RGBC-WS2812B, RevK:SMD1010, F.Cu at (56.7, 129.6)
- added D170: XL-1010RGBC-WS2812B, RevK:SMD1010, F.Cu at (52.7, 122.7)
- added D171: XL-1010RGBC-WS2812B, RevK:SMD1010, F.Cu at (47.8, 94.8)
- added D172: XL-1010RGBC-WS2812B, RevK:SMD1010, F.Cu at (49.1, 87.0)
- added D173: XL-1010RGBC-WS2812B, RevK:SMD1010, F.Cu at (63.3, 62.5)
- added D174: XL-1010RGBC-WS2812B, RevK:SMD1010, F.Cu at (69.4, 57.3)
- added D175: XL-1010RGBC-WS2812B, RevK:SMD1010, F.Cu at (95.0, 45.2)
- added D176: XL-1010RGBC-WS2812B, RevK:SMD1010, F.Cu at (105.0, 45.2)
- added D177: XL-1010RGBC-WS2812B, RevK:SMD1010, F.Cu at (131.4, 54.8)
- added D178: XL-1010RGBC-WS2812B, RevK:SMD1010, F.Cu at (139.0, 61.3)
- added D179: XL-1010RGBC-WS2812B, RevK:SMD1010, F.Cu at (153.1, 85.6)
- added D180: XL-1010RGBC-WS2812B, RevK:SMD1010, F.Cu at (154.8, 95.4)
- added D181: XL-1010RGBC-WS2812B, RevK:SMD1010, F.Cu at (149.9, 123.1)
- added D182: XL-1010RGBC-WS2812B, RevK:SMD1010, F.Cu at (144.9, 131.7)
- added D183: XL-1010RGBC-WS2812B, RevK:SMD1010, F.Cu at (123.4, 149.8)
- added D184: XL-1010RGBC-WS2812B, RevK:SMD1010, F.Cu at (114.0, 153.2)
- added D185: XL-1010RGBC-WS2812B, RevK:SMD1010, F.Cu at (86.0, 153.2)
- added D186: XL-1010RGBC-WS2812B, RevK:SMD1010, F.Cu at (76.6, 149.8)
- added D187: XL-1010RGBC-WS2812B, RevK:SMD1010, F.Cu at (55.1, 131.7)
- added D188: XL-1010RGBC-WS2812B, RevK:SMD1010, F.Cu at (50.1, 123.1)
- added D189: XL-1010RGBC-WS2812B, RevK:SMD1010, F.Cu at (45.2, 95.4)
- added D190: XL-1010RGBC-WS2812B, RevK:SMD1010, F.Cu at (46.9, 85.6)
- added D191: XL-1010RGBC-WS2812B, RevK:SMD1010, F.Cu at (61.0, 61.3)
- added D192: XL-1010RGBC-WS2812B, RevK:SMD1010, F.Cu at (68.6, 54.8)
- added D193: XL-1010RGBC-WS2812B, RevK:SMD1010, F.Cu at (94.0, 42.8)
- added D194: XL-1010RGBC-WS2812B, RevK:SMD1010, F.Cu at (106.0, 42.8)
- added D195: XL-1010RGBC-WS2812B, RevK:SMD1010, F.Cu at (132.2, 52.3)
- added D196: XL-1010RGBC-WS2812B, RevK:SMD1010, F.Cu at (141.3, 60.0)
- added D197: XL-1010RGBC-WS2812B, RevK:SMD1010, F.Cu at (155.3, 84.2)
- added D198: XL-1010RGBC-WS2812B, RevK:SMD1010, F.Cu at (157.4, 96.0)
- added D199: XL-1010RGBC-WS2812B, RevK:SMD1010, F.Cu at (152.5, 123.4)
- added D200: XL-1010RGBC-WS2812B, RevK:SMD1010, F.Cu at (146.5, 133.8)
- added D201: XL-1010RGBC-WS2812B, RevK:SMD1010, F.Cu at (125.2, 151.7)
- added D202: XL-1010RGBC-WS2812B, RevK:SMD1010, F.Cu at (113.9, 155.8)
- added D203: XL-1010RGBC-WS2812B, RevK:SMD1010, F.Cu at (86.1, 155.8)
- added D204: XL-1010RGBC-WS2812B, RevK:SMD1010, F.Cu at (74.8, 151.7)
- added D205: XL-1010RGBC-WS2812B, RevK:SMD1010, F.Cu at (53.5, 133.8)
- added D206: XL-1010RGBC-WS2812B, RevK:SMD1010, F.Cu at (47.5, 123.4)
- added D207: XL-1010RGBC-WS2812B, RevK:SMD1010, F.Cu at (42.6, 96.0)
- added D208: XL-1010RGBC-WS2812B, RevK:SMD1010, F.Cu at (44.7, 84.2)
- added D209: XL-1010RGBC-WS2812B, RevK:SMD1010, F.Cu at (58.7, 60.0)
- added D210: XL-1010RGBC-WS2812B, RevK:SMD1010, F.Cu at (67.8, 52.3)
- added J1: Conn_01x03, RevK:3-PADS, B.Cu at (104.2, 44.8)
- added J2: Conn_01x03, RevK:3-PADS, B.Cu at (100.3, 44.8)
Connections:
- D1 pad 4: unconnected-(D1-I-Pad4) -> Net-(D1-I)
- D117 pad 1: unconnected-(D117-O-Pad1) -> Net-(D117-O)
Routing:
- net GND: track 0.00 -> 1695.3 mm, vias 0 -> 5
- net VCC: track 0.00 -> 1661.4 mm, vias 0 -> 5
- net (no net): track 800.0 -> 0.00 mm, vias 2 -> 0
- net Net-(D210-O): track 0.00 -> 46.3 mm, vias 0 -> 1
- net Net-(D192-O): track 0.00 -> 31.9 mm, vias 0 -> 2
- net Net-(D174-O): track 0.00 -> 31.6 mm, vias 0 -> 2
- net Net-(D117-O): track 0.00 -> 30.0 mm, vias 0 -> 2
- net Net-(D172-O): track 0.00 -> 27.4 mm
- net Net-(D160-O): track 0.00 -> 27.4 mm
- net Net-(D166-O): track 0.00 -> 27.4 mm
- net Net-(D170-O): track 0.00 -> 27.4 mm
- net Net-(D162-O): track 0.00 -> 27.4 mm
- net Net-(D164-O): track 0.00 -> 27.4 mm
- net Net-(D168-O): track 0.00 -> 27.4 mm
- net Net-(D158-O): track 0.00 -> 27.4 mm
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- added copper zone on B.Cu, net GND

Commit message: Needs more work
Parts:
- Logo1, U1: moved to B.Cu
- moved Logo1 55.9 mm to (45.0, 100.0), turned to 180 degrees
- moved U1 55.0 mm to (155.0, 100.0), turned to 180 degrees

Commit message: Tidy
Parts:
- moved J2 111.7 mm to (97.0, 156.5)
- moved J1 111.7 mm to (103.0, 156.5)
Routing:
- net Net-(D1-I): track 13.4 -> 198.4 mm
- net Net-(D210-O): track 46.3 -> 214.2 mm
- net GND: track 1695.3 -> 1816.9 mm, vias 5 -> 207
- net VCC: track 1661.4 -> 1744.2 mm, vias 5 -> 202
- net Net-(D117-O): track 30.0 -> 15.7 mm
- net Net-(D156-O): track 10.2 -> 17.0 mm
- net Net-(D174-O): track 31.6 -> 33.9 mm
- net Net-(D192-O): track 31.9 -> 33.7 mm
- added copper zone on B.Cu, net VCC
Other:
- board text added: "${CURRENT_DATE}"
