File: PCB/LEDX/LEDX.kicad_sch (KiCad schematic)
At the start: 22 parts, among them J2 Conn_01x03, J3 TC2030-USB-NL-DS, U1 ICS43434_MEMS_Mic, U2 ESP32-S3-MINI-1, U5 MD8942

Commit message: Started
Parts:
- added C5: 100nF, RevK:C_0402, symbol Device:C
- added U3: 78L05, RevK:SOT-23, symbol RevK:78L05
Connections:
- net +3.3V: no longer D1.2 (+)
- net DC: now also U3.2 (IN)
- net GND: now also C5.1, U3.3 (GND)
- net at D1.1 (O): now also D2.2, J2.2 (Pin_2)
- net LED1 renamed LED
- removed net LED2: D2.2, J2.2 (Pin_2), U2.5 (GPIO1)
- new net: C5.2, D1.2 (+), U3.1 (OUT)
Other:
- moved on the sheet: C4, D1, D2

Commit message: Tracked
Connections:
- net +3.3V: now also U2.29 (GPIO34); no longer U2.18 (GPIO14)
- net SCK: now also U2.30 (GPIO48); no longer U2.19 (GPIO15)
- net SD: now also U2.28 (GPIO33); no longer U2.17 (GPIO13)
- net WS: now also U2.25 (GPIO21); no longer U2.16 (GPIO12)
- no-connect marks 32 -> 28
Changed lines of the file:
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@@
-	)
-	(no_connect
-		(at 124.46 67.945)
 	)
 	(no_connect
@@
 	)
 	(no_connect
-		(at 124.46 103.505)
-	)
-	(no_connect
 		(at 74.93 40.005)
 	)
 	(no_connect
-		(at 124.46 70.485)
-	)
-	(no_connect
 		(at 124.46 90.805)
 	)
@@
 	(no_connect
 		(at 124.46 88.265)
-	)
-	(no_connect
-		(at 93.98 103.505)
 	)
 	(no_connect
@@
 	(global_label "WS"
 		(shape output)
-		(at 93.98 80.645 180)
+		(at 93.98 103.505 180)
 		(fields_autoplaced yes)
 		(effects
@@
 		)
 		(property "Intersheetrefs" "${INTERSHEET_REFS}"
-			(at 88.9881 80.645 0)
+			(at 88.9881 103.505 0)
 			(effects
 				(font
@@
 	(global_label "SD"
 		(shape input)
-		(at 93.98 83.185 180)
+		(at 124.46 67.945 0)
 		(fields_autoplaced yes)
 		(effects
@@
 				(size 1.27 1.27)
 			)
-			(justify right)
+			(justify left)
 		)
 		(property "Intersheetrefs" "${INTERSHEET_REFS}"
-			(at 89.1695 83.185 0)
-			(effects
-				(font
-					(size 1.27 1.27)
-				)
-				(justify right)
+			(at 129.2705 67.945 0)
+			(effects
+				(font
+					(size 1.27 1.27)
+				)
+				(justify left)
 				(hide yes)
 			)
@@
 	(global_label "SCK"
 		(shape output)
-		(at 93.98 88.265 180)
+		(at 124.46 103.505 0)
 		(fields_autoplaced yes)
 		(effects
@@
 				(size 1.27 1.27)
 			)
-			(justify right)
+			(justify left)
 		)
 		(property "Intersheetrefs" "${INTERSHEET_REFS}"
-			(at 87.8995 88.265 0)
-			(effects
-				(font
-					(size 1.27 1.27)
-				)
-				(justify right)
+			(at 130.5405 103.505 0)
+			(effects
+				(font
+					(size 1.27 1.27)
+				)
+				(justify left)
 				(hide yes)
 			)
@@
 	(symbol
 		(lib_id "power:+3.3V")
-		(at 93.98 85.725 90)
+		(at 124.46 70.485 270)
 		(unit 1)
 		(exclude_from_sim no)
@@
 		(fields_autoplaced yes)
 		(property "Reference" "#PWR04"
-			(at 97.79 85.725 0)
+			(at 120.65 70.485 0)
 			(effects
 				(font
@@
 		)
 		(property "Value" "+3.3V"
-			(at 90.805 85.725 90)
+			(at 127.635 70.485 90)
 			(effects
 				(font
@@
 		)
 		(property "Footprint" ""
-			(at 93.98 85.725 0)
+			(at 124.46 70.485 0)
 			(effects
 				(font
@@
 		)
 		(property "Datasheet" ""
-			(at 93.98 85.725 0)
+			(at 124.46 70.485 0)
 			(effects
 				(font
@@
 		)
 		(property "Description" "Power symbol creates a global label with name \"+3.3V\""
-			(at 93.98 85.725 0)
-			(effects
-				(font
+			(at 124.46 70.485 0)
+			(effects
+				(font

Commit message: Limitation
Other:
- note added: "This only works for RGB not RGBW"
Changed lines of the file:
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@@
+		)
+	)
+	(text "This only works for RGB not RGBW"
+		(exclude_from_sim no)
+		(at 146.05 137.922 0)
+		(effects
+			(font
+				(size 12.7 12.7)
+			)
 		)
 	)

Commit message: Not level convert as fixes to RGB mode
Parts:
- removed C5: 100nF, RevK:C_0402, symbol Device:C
- removed U3: 78L05, RevK:SOT-23, symbol RevK:78L05
Connections:
- net +3.3V: now also D1.2 (+)
- net LED1: now reaches D2.2, J2.2 (Pin_2)
- net LED1: now also U2.5 (GPIO1); no longer D1.1 (O)
- net LED renamed LED2
- no-connect marks 28 -> 30
Other:
- note removed: "This only works for RGB not RGBW"
- title: Generic ESP32 USB-A -> LED driver
- moved on the sheet: D1

Commit message: Pads
Parts:
- added P1, P2, P3, P4: Square, RevK:PAD-2mm, symbol RevK:SquareSMD
Connections:
- net D+: now also P3.1 (P)
- net D-: now also P2.1 (P)
- net DC: now also P1.1 (P)
- net GND: now also P4.1 (P)

Commit message: Tidy
Changed lines of the file:
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@@
 	(global_label "D+"
 		(shape bidirectional)
-		(at 240.665 108.585 0)
+		(at 240.665 109.855 0)
 		(fields_autoplaced yes)
 		(effects
@@
 		)
 		(property "Intersheetrefs" "${INTERSHEET_REFS}"
-			(at 246.7909 108.585 0)
+			(at 246.7909 109.855 0)
 			(effects
 				(font
@@
 	(symbol
 		(lib_id "power:GND")
-		(at 240.665 112.395 90)
+		(at 240.665 113.665 90)
 		(unit 1)
 		(exclude_from_sim no)
@@
 		(fields_autoplaced yes)
 		(property "Reference" "#PWR07"
-			(at 247.015 112.395 0)
+			(at 247.015 113.665 0)
 			(effects
 				(font
@@
 		)
 		(property "Value" "GND"
-			(at 243.84 112.395 90)
+			(at 243.84 113.665 90)
 			(effects
 				(font
@@
 		)
 		(property "Footprint" ""
-			(at 240.665 112.395 0)
+			(at 240.665 113.665 0)
 			(effects
 				(font
@@
 		)
 		(property "Datasheet" ""
-			(at 240.665 112.395 0)
+			(at 240.665 113.665 0)
 			(effects
 				(font
@@
 		)
 		(property "Description" "Power symbol creates a global label with name \"GND\" , ground"
-			(at 240.665 112.395 0)
+			(at 240.665 113.665 0)
 			(effects
 				(font
@@
 	(symbol
 		(lib_id "RevK:SquareSMD")
-		(at 240.665 108.585 180)
+		(at 240.665 109.855 180)
 		(unit 1)
 		(exclude_from_sim no)
@@
 		(dnp no)
 		(property "Reference" "P3"
-			(at 234.315 108.585 0)
+			(at 234.315 109.855 0)
 			(effects
 				(font
@@
 		)
 		(property "Value" "Square"
-			(at 233.68 108.458 0)
+			(at 233.68 109.728 0)
 			(effects
 				(font
@@
 		)
 		(property "Footprint" "RevK:PAD-2mm"
-			(at 240.665 106.045 0)
+			(at 240.665 107.315 0)
 			(effects
 				(font
@@
 		)
 		(property "Datasheet" ""
-			(at 240.665 108.585 0)
+			(at 240.665 109.855 0)
 			(effects
 				(font
@@
 		)
 		(property "Description" ""
-			(at 240.665 108.585 0)
+			(at 240.665 109.855 0)
 			(effects
 				(font
@@
 	(symbol
 		(lib_id "RevK:SquareSMD")
-		(at 240.665 112.395 180)
+		(at 240.665 113.665 180)
 		(unit 1)
 		(exclude_from_sim no)
@@
 		(dnp no)
 		(property "Reference" "P4"
-			(at 234.315 112.395 0)
+			(at 234.315 113.665 0)
 			(effects
 				(font
@@
 		)
 		(property "Value" "Square"
-			(at 233.68 112.268 0)
+			(at 233.68 113.538 0)
 			(effects
 				(font
@@
 		)
 		(property "Footprint" "RevK:PAD-2mm"
-			(at 240.665 109.855 0)
+			(at 240.665 111.125 0)
 			(effects
 				(font
@@
 		)
 		(property "Datasheet" ""
-			(at 240.665 112.395 0)
+			(at 240.665 113.665 0)
 			(effects
 				(font
@@
 		)
 		(property "Description" ""
-			(at 240.665 112.395 0)
+			(at 240.665 113.665 0)
 			(effects
 				(font
