File: PCB/Coaster2/Coaster.kicad_pcb (KiCad board)
At the start: 2 copper layers, 100 x 100 mm, 278 parts, among them J2 TC2030-USB-NL-DS, J3 USB-C-Socket-H, U1 ICS43434_MEMS_Mic, U2 ESP32-S3-MINI-1, U3 MD8942

Commit message: SS
Parts:
- added J1: Reset, RevK:AA-Pad, B.Cu at (100.0, 100.0)
Connections:
- U2 pad 25: unconnected-(U2-GPIO21-Pad25) -> Net-(J1-Pin_2)
Routing:
- net Net-(J1-Pin_2): track 0.00 -> 7.05 mm, vias 0 -> 1
Other:
- board text added: "124 LEDs 4+8+16+32+64"
- board text added: "21"
- board text added: "37 40 41 42"
- board text added: "LED WS SD SCK"

Commit message: Tidy
Routing:
- net Net-(J3-CC2): track 5.74 -> 8.13 mm
- net Net-(J3-CC1): track 6.08 -> 8.47 mm

Commit message: Final, and spacers
Parts:
- removed FID1, FID2, FID3: Fiducial, RevK:Hole-Tooling
- removed FID4, FID5, FID6: Fiducial, Fiducial:Fiducial_1mm_Mask2mm
- added PCB1: 120x120, RevK:PCB120120, F.Cu at (100.0, 100.0)
- added V1: ~, RevK:VCUT120N, F.Cu at (100.0, 50.1)
- added V2: ~, RevK:VCUT120N, F.Cu at (100.0, 149.9)
- added V3: ~, RevK:VCUT120N, F.Cu at (149.9, 100.0)
- added V4: ~, RevK:VCUT120N, F.Cu at (50.1, 100.0)
Other:
- board size 100 x 100 mm -> 120 x 120 mm
- board text added: "37"
- board text added: "40 41 42"
- board text added: "LED"
- board text added: "WS SD SCK"
- board text removed: "37 40 41 42"
- board text removed: "LED WS SD SCK"

Commit message: Tidy
Routing:
- net GND: track 1086.1 -> 1099.9 mm, vias 143 -> 144
- net VBUS: track 1079.4 -> 1079.2 mm, vias 128 -> 131
