File: PCB/Coaster2/Spacer.kicad_pcb (KiCad board)
At the start: 2 copper layers, 99.7 x 100 mm, 1 part

Commit message: tidy
Routing:
- removed copper zone on F.Cu, net GND
Changed lines of the file:
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@@
 	)
 	(net 0 "")
-	(net 1 "GND")
 	(footprint "RevK:Shadow"
 		(layer "F.Cu")
@@
 		(layer "Edge.Cuts")
 	)
-	(zone
-		(net 1)
-		(net_name "GND")
-		(layer "F.Cu")
-		(hatch edge 0.5)
-		(priority 3)
-		(connect_pads
-			(clearance 0.127)
-		)
-		(min_thickness 0.25)
-		(filled_areas_thickness no)
-		(fill yes
-			(thermal_gap 0.5)
-			(thermal_bridge_width 0.5)
-		)
-		(polygon
-			(pts
-				(xy 150 95) (xy 141 95) (xy 141 105) (xy 150 105)
-			)
-		)
-	)
 )
