File: PCB/LED32/LED.kicad_sch (KiCad schematic)
At the start: 178 parts, among them P1 Square, P2 Square, P3 Square

Commit message: Re-image
Parts:
- added C88: 100nF, RevK:C_0402, symbol Device:C
Connections:
- net GND: now also C88.2
- net VCC: now also C88.1
Changed lines of the file:
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@@
 	)
 	(junction
+		(at 107.315 124.46)
+		(diameter 0)
+		(color 0 0 0 0)
+	)
+	(junction
 		(at 103.505 125.095)
 		(diameter 0)
@@
 	)
 	(junction
-		(at 107.315 118.745)
-		(diameter 0)
-		(color 0 0 0 0)
-	)
-	(junction
 		(at 46.355 61.595)
 		(diameter 0)
@@
 	)
 	(junction
+		(at 107.315 118.745)
+		(diameter 0)
+		(color 0 0 0 0)
+	)
+	(junction
 		(at 107.315 106.045)
 		(diameter 0)
@@
 	)
 	(junction
+		(at 114.935 118.745)
+		(diameter 0)
+		(color 0 0 0 0)
+	)
+	(junction
 		(at 92.075 125.095)
 		(diameter 0)
@@
 	(wire
 		(pts
+			(xy 107.315 118.745) (xy 107.315 124.46)
+		)
+		(stroke
+			(width 0)
+			(type default)
+		)
+	)
+	(wire
+		(pts
 			(xy 46.355 86.995) (xy 46.355 93.345)
 		)
@@
 	(wire
 		(pts
+			(xy 114.935 118.745) (xy 114.935 124.46)
+		)
+		(stroke
+			(width 0)
+			(type default)
+		)
+	)
+	(wire
+		(pts
 			(xy 99.695 97.155) (xy 99.695 102.235)
 		)
@@
 	(symbol
 		(lib_id "power:GND")
-		(at 107.315 118.745 0)
+		(at 107.315 124.46 0)
 		(unit 1)
 		(exclude_from_sim no)
@@
 		(fields_autoplaced yes)
 		(property "Reference" "#PWR09"
-			(at 107.315 125.095 0)
+			(at 107.315 130.81 0)
 			(effects
 				(font
@@
 		)
 		(property "Value" "GND"
-			(at 107.315 122.8781 0)
+			(at 107.315 128.5931 0)
 			(effects
 				(font
@@
 		)
 		(property "Footprint" ""
-			(at 107.315 118.745 0)
+			(at 107.315 124.46 0)
 			(effects
 				(font
@@
 		)
 		(property "Datasheet" ""
-			(at 107.315 118.745 0)
+			(at 107.315 124.46 0)
 			(effects
 				(font
@@
 		)
 		(property "Description" "Power symbol creates a global label with name \"GND\" , ground"
-			(at 107.315 118.745 0)
+			(at 107.315 124.46 0)
 			(effects
 				(font
@@
 					(unit 1)
 				)
+			)
+		)
+	)
+	(symbol
+		(lib_id "Device:C")
+		(at 111.125 124.46 270)
+		(mirror x)
+		(unit 1)
+		(exclude_from_sim no)
+		(in_bom yes)
+		(on_board yes)
+		(dnp no)
+		(property "Reference" "C88"
+			(at 113.03 124.46 0)
+			(effects
+				(font
+					(size 1 1)
+				)
+			)
+		)
+		(property "Value" "100nF"
+			(at 111.125 124.46 0)
+			(effects
+				(font
+					(size 1 1)
+				)
+			)
+		)
+		(property "Footprint" "RevK:C_0402"
+			(at 107.315 123.4948 0)
+			(effects
+				(font
+					(size 1.27 1.27)
+				)
+				(hide yes)
+			)
+		)
+		(property "Datasheet" "~"
+			(at 111.125 124.46 0)
+			(effects
+				(font
+					(size 1.27 1.27)
+				)
+				(hide yes)
+			)
+		)
+		(property "Description" "Unpolarized capacitor"
+			(at 111.125 124.46 0)
+			(effects
+				(font
+					(size 1.27 1.27)
+				)
+				(hide yes)
+			)
+		)
+		(pin "1"
+		)
+		(pin "2"
+		)
+		(instances
+			(project "LED"
+				(path "/46c350bb-7de4-4e81-aafd-4af55e37aab0"
+					(reference "C88")
+					(unit 1)
+				)

Commit message: PCB Update
Parts:
- D1, D10, D11, D12, D13, D14, D15, D16, D17, D18, D19, D2, D20, D21, D22, D23, D24, D25, D26, D27, D28, D29, D3, D30, D31, D32, D33, D34, D35, D36, D37, D38, D39, D4, D40, D41, D42, D43, D44, D45, D46, D47, D48, D49, D5, D50, D51, D52, D53, D54, D55, D56, D57, D58, D59, D6, D60, D61, D62, D63, D64, D65, D66, D67, D68, D69, D7, D70, D71, D72, D73, D74, D75, D76, D77, D78, D79, D8, D80, D81, D82, D83, D84, D85, D86, D87, D88, D9: LCSC Part # C5349953 -> (none); MPN (none) -> C5349953
