File: PCB/LED32/LED.kicad_pcb (KiCad board)
At the start: 2 copper layers, 32 x 32 mm, 178 parts, among them P1 Square, P2 Square, P3 Square

Commit message: Re-image
Parts:
- added C88: 100nF, RevK:C_0402, F.Cu at (98.6, 86.1)
Routing:
- net VCC: track 297.1 -> 315.4 mm
- net GND: track 315.6 -> 333.2 mm
- net Net-(D56-O): track 4.38 -> 5.53 mm

Commit message: Images
Parts:
- moved P3 6.10 mm to (97.5, 102.0)
- moved P1 2.69 mm to (102.5, 98.0)
Routing:
- net VCC: track 315.4 -> 318.7 mm
- net GND: track 333.2 -> 335.2 mm
