File: PCB/Coaster3/Coaster.kicad_sch (KiCad schematic)
At the start: 279 parts, among them J1 Reset, J2 TC2030-USB-NL-DS, J3 USB-C-Socket-H, J4 DC, J5 DC, U1 ICS43434_MEMS_Mic, U2 ESP32-S3-MINI-1, U3 MD8942

Commit message: Library update
Parts:
- removed C129: 100nF, RevK:C_0402, symbol Device:C
- removed C130: 22uF, RevK:C_0603, symbol Device:C
- removed C137: 10uF 35V, RevK:C_0603_, symbol RevK:Hidden
- removed C138: 10uF 6.3V, RevK:C_0603_, symbol RevK:Hidden
- removed C139: 100nF, RevK:C_0603_, symbol RevK:Hidden
- removed L1: 10uH, RevK:L_4x4_, symbol RevK:Hidden
- removed R2: 124k, RevK:R_0402_, symbol RevK:Hidden
- removed R3: 39k2, RevK:R_0402_, symbol RevK:Hidden
- removed R4: 1M, RevK:R_0402_, symbol RevK:Hidden
- removed U3: MD8942, RevK:SOT-23-6-MD8942, symbol RevK:MD89420-RegBlock
- added C133: 22uF 25V, RevK:C_0805, symbol Device:C
- added C134, C135: 100nF 25V, RevK:C_0402, symbol Device:C
- added C137: 18pF, RevK:C_0201, symbol Device:C
- added C138: 47uF 6V, RevK:C_0805, symbol Device:C
- added C139, C140, C141: 100nF, RevK:C_0201, symbol Device:C
- added L1: 4.7uH, RevK:L_5x5, symbol Device:L
- added R4, R5: 150k 1%, RevK:R_0201, symbol Device:R
- added R6: 33k 1%, RevK:R_0201, symbol Device:R
- added U3: TPS562246, RevK:SOT-563, symbol RevK:TPS562246
- C1, C10, C100, C101, C102, C103, C104, C105, C106, C107, C108, C109, C11, C110, C111, C112, C113, C114, C115, C116, C117, C118, C119, C12, C120, C121, C122, C123, C124, C13, C14, C15, C16, C17, C18, C19, C2, C20, C21, C22, C23, C24, C25, C26, C27, C28, C29, C3, C30, C31, C32, C33, C34, C35, C36, C37, C38, C39, C4, C40, C41, C42, C43, C44, C45, C46, C47, C48, C49, C5, C50, C51, C52, C53, C54, C55, C56, C57, C58, C59, C6, C60, C61, C62, C63, C64, C65, C66, C67, C68, C69, C7, C70, C71, C72, C73, C74, C75, C76, C77, C78, C79, C8, C80, C81, C82, C83, C84, C85, C86, C87, C88, C89, C9, C90, C91, C92, C93, C94, C95, C96, C97, C98, C99: footprint RevK:C_0402 -> RevK:C_0201
- C128: renamed from C132; footprint RevK:C_0402 -> RevK:C_0201
- C130: renamed from C134; footprint RevK:C_0402 -> RevK:C_0201
- C136: value 10uF 35V -> 100nF; footprint RevK:C_0603 -> RevK:C_0201; MPN C194427 -> C76934
- R1: footprint RevK:R_0402 -> RevK:R_0201
- R2: renamed from R5; footprint RevK:R_0402 -> RevK:R_0201
- R3: renamed from R6; footprint RevK:R_0402 -> RevK:R_0201
- renumbered C131 to C127, C133 to C129, C135 to C131, J4 to J2, J5 to J3, J2 to J4, J3 to J5, V4 to V1, V1 to V2, V2 to V3, V3 to V4
Connections:
- net +3V3: now also C137.2, C138.1, C139.2, C140.2, C141.2, L1.2, R5.1; no longer C136.1
- net GND: now also C133.2, C134.2, C135.2, C138.2, C139.1, C140.1, C141.1, R6.2, U3.3 (GND); no longer C136.2
- net VBUS: now also C29.1, C30.1, D30.3 (+), C133.1, C134.1, C135.1, R4.2, U3.1 (VIN)
- new net BST: C136.1, U3.4 (VBST)
- new net EN: R4.1, U3.5 (EN)
- new net FB: C137.1, R5.2, R6.1, U3.6 (VFB)
- new net SW: C136.2, L1.1, U3.2 (SW)
- no-connect marks 32 -> 31
