File: PCB/Test/LED.kicad_pcb (KiCad board)
At the start: 2 copper layers, 25 x 45 mm, 45 parts

Commit message: Spacing
Parts:
- moved D40 0.90 mm to (107.5, 92.7)
- moved D39 0.80 mm to (107.5, 94.9)
- moved D38 0.70 mm to (107.5, 97.1)
- moved D37 0.60 mm to (107.5, 99.3)
- moved D36 0.50 mm to (107.5, 101.5)
- moved D35 0.40 mm to (107.5, 103.7)
- moved D34 0.30 mm to (107.5, 105.9)
- moved D33 0.20 mm to (107.5, 108.1)
- moved D32 0.10 mm to (107.5, 110.3)
Routing:
- net +3V3: track 33.2 -> 32.6 mm
Changed lines of the file:
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@@
 	(footprint "RevK:SMD2020"
 		(layer "F.Cu")
-		(at 107.5 95.7 180)
+		(at 107.5 94.9 180)
 		(descr "https://cdn-shop.adafruit.com/datasheets/WS2812B.pdf")
 		(tags "LED RGB NeoPixel")
@@
 	(footprint "RevK:SMD2020"
 		(layer "F.Cu")
-		(at 107.5 97.8 90)
+		(at 107.5 97.1 90)
 		(descr "https://cdn-shop.adafruit.com/datasheets/WS2812B.pdf")
 		(tags "LED RGB NeoPixel")
@@
 	(footprint "RevK:SMD2020"
 		(layer "F.Cu")
-		(at 107.5 104.1 180)
+		(at 107.5 103.7 180)
 		(descr "https://cdn-shop.adafruit.com/datasheets/WS2812B.pdf")
 		(tags "LED RGB NeoPixel")
@@
 	(footprint "RevK:SMD2020"
 		(layer "F.Cu")
-		(at 107.5 108.3 180)
+		(at 107.5 108.1 180)
 		(descr "https://cdn-shop.adafruit.com/datasheets/WS2812B.pdf")
 		(tags "LED RGB NeoPixel")
@@
 	(footprint "RevK:SMD2020"
 		(layer "F.Cu")
-		(at 107.5 106.2 90)
+		(at 107.5 105.9 90)
 		(descr "https://cdn-shop.adafruit.com/datasheets/WS2812B.pdf")
 		(tags "LED RGB NeoPixel")
@@
 	(footprint "RevK:SMD2020"
 		(layer "F.Cu")
-		(at 107.5 93.6 90)
+		(at 107.5 92.7 90)
 		(descr "https://cdn-shop.adafruit.com/datasheets/WS2812B.pdf")
 		(tags "LED RGB NeoPixel")
@@
 	(footprint "RevK:SMD2020"
 		(layer "F.Cu")
-		(at 107.5 102 90)
+		(at 107.5 101.5 90)
 		(descr "https://cdn-shop.adafruit.com/datasheets/WS2812B.pdf")
 		(tags "LED RGB NeoPixel")
@@
 	(footprint "RevK:SMD2020"
 		(layer "F.Cu")
-		(at 107.472659 99.902352 180)
+		(at 107.5 99.3 180)
 		(descr "https://cdn-shop.adafruit.com/datasheets/WS2812B.pdf")
 		(tags "LED RGB NeoPixel")
@@
 	(footprint "RevK:SMD2020"
 		(layer "F.Cu")
-		(at 107.5 110.4 90)
+		(at 107.5 110.3 90)
 		(descr "https://cdn-shop.adafruit.com/datasheets/WS2812B.pdf")
 		(tags "LED RGB NeoPixel")
@@
 	)
 	(segment
-		(start 98.1 92)
-		(end 98.1 95.749)
+		(start 103.175 89.46)
+		(end 107.221364 89.46)
 		(width 1)
 		(layer "F.Cu")
@@
 	)
 	(segment
-		(start 94 89.5)
-		(end 92.75 88.25)
+		(start 98.1 92)
+		(end 98.1 95.749)
 		(width 1)
 		(layer "F.Cu")
@@
 	)
 	(segment
-		(start 103.175 89.46)
-		(end 106.321364 89.46)
+		(start 94 89.5)
+		(end 92.75 88.25)
 		(width 1)
 		(layer "F.Cu")
@@
 	)
 	(segment
-		(start 106.321364 89.46)
-		(end 109.116 92.254636)
-		(width 1)
-		(layer "F.Cu")
-		(net 2)
-	)
-	(segment
 		(start 94 94)
 		(end 94 89.5)
@@
 	)
 	(segment
+		(start 107.221364 89.46)
+		(end 108.980682 91.219318)
+		(width 1)
+		(layer "F.Cu")
+		(net 2)
+	)
+	(segment
 		(start 101.116 88.384)
 		(end 98.1 91.4)
@@
 	(segment
 		(start 106.825 111.96)
-		(end 106.825 111.21)
+		(end 106.825 111.11)
 		(width 0.25)
 		(layer "F.Cu")
@@
 	)
 	(segment
-		(start 108.04 109.725)
-		(end 108.04 108.975)
+		(start 108.175 108.64)
+		(end 108.175 109.49)
 		(width 0.25)
 		(layer "F.Cu")
@@
 	)
 	(segment
-		(start 106.825 107.76)
-		(end 106.825 107.01)
+		(start 106.96 106.575)
+		(end 106.96 107.425)
 		(width 0.25)
 		(layer "F.Cu")
@@
 	)
 	(segment
-		(start 108.04 105.525)
-		(end 108.04 104.775)
+		(start 108.04 105.225)
+		(end 108.04 104.375)
 		(width 0.25)
 		(layer "F.Cu")
@@
 	)
 	(segment
-		(start 106.825 103.56)
-		(end 106.825 102.81)
+		(start 106.825 103.16)
+		(end 106.825 102.31)
 		(width 0.25)
 		(layer "F.Cu")
@@
 	)
 	(segment
-		(start 108.04 101.325)
-		(end 108.04 100.550011)
+		(start 108.04 100.825)
+		(end 108.04 99.975)
 		(width 0.25)
 		(layer "F.Cu")
@@
 	)
 	(segment
-		(start 106.797659 99.362352)
-		(end 106.797659 98.637341)
+		(start 106.825 98.76)
+		(end 106.825 97.91)
 		(width 0.25)
 		(layer "F.Cu")
@@
 	)
 	(segment
-		(start 108.04 97.125)
-		(end 108.04 96.375)
+		(start 108.04 96.425)
+		(end 108.04 95.575)
 		(width 0.25)
 		(layer "F.Cu")
@@
 	)
 	(segment
-		(start 106.825 95.16)
-		(end 106.825 94.41)
+		(start 106.825 94.36)
+		(end 106.825 93.51)
 		(width 0.25)
 		(layer "F.Cu")
@@
 		(polygon
 			(pts
-				(xy 107.5 114) (xy 107.5 92.1) (xy 109.5 92.1) (xy 109.5 114)
+				(xy 107.5 114) (xy 107.5 91) (xy 109.5 91) (xy 109.5 114)
 			)
 		)

Commit message: Tweaked design
Parts:
- D11, D12, D13, D14, D15, D16, D17, D18, D19, D20: value XL-1010RGBC-WS2812B -> XL-1615RGBC-WS2812B
- D21, D22, D23, D24, D25, D26, D27, D28, D29, D30, D31, D32, D33, D34, D35, D36, D37, D38, D39, D40: value XL-1010RGBC-WS2812B -> XL-2020RGBC-WS2812B
Changed lines of the file:
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@@
 			)
 		)
-		(property "Value" "XL-1010RGBC-WS2812B"
+		(property "Value" "XL-2020RGBC-WS2812B"
 			(at 0 2.25 0)
 			(layer "F.Fab")
@@
 			)
 		)
-		(property "Value" "XL-1010RGBC-WS2812B"
+		(property "Value" "XL-2020RGBC-WS2812B"
 			(at 0 2.25 0)
 			(layer "F.Fab")
@@
 			)
 		)
-		(property "Value" "XL-1010RGBC-WS2812B"
+		(property "Value" "XL-1615RGBC-WS2812B"
 			(at 0 2.25 0)
 			(layer "F.Fab")
@@
 			)
 		)
-		(property "Value" "XL-1010RGBC-WS2812B"
+		(property "Value" "XL-2020RGBC-WS2812B"
 			(at 0 2.25 0)
 			(layer "F.Fab")
@@
 			)
 		)
-		(property "Value" "XL-1010RGBC-WS2812B"
+		(property "Value" "XL-2020RGBC-WS2812B"
 			(at 0 2.25 0)
 			(layer "F.Fab")
@@
 			)
 		)
-		(property "Value" "XL-1010RGBC-WS2812B"
+		(property "Value" "XL-2020RGBC-WS2812B"
 			(at 0 2.25 0)
 			(layer "F.Fab")
@@
 			)
 		)
-		(property "Value" "XL-1010RGBC-WS2812B"
+		(property "Value" "XL-2020RGBC-WS2812B"
 			(at 0 2.25 0)
 			(layer "F.Fab")
@@
 			)
 		)
-		(property "Value" "XL-1010RGBC-WS2812B"
+		(property "Value" "XL-1615RGBC-WS2812B"
 			(at 0 2.25 0)
 			(layer "F.Fab")
@@
 			)
 		)
-		(property "Value" "XL-1010RGBC-WS2812B"
+		(property "Value" "XL-1615RGBC-WS2812B"
 			(at 0 2.25 0)
 			(layer "F.Fab")
@@
 			)
 		)
-		(property "Value" "XL-1010RGBC-WS2812B"
+		(property "Value" "XL-2020RGBC-WS2812B"
 			(at 0 2.25 90)
 			(layer "F.Fab")
@@
 			)
 		)
-		(property "Value" "XL-1010RGBC-WS2812B"
+		(property "Value" "XL-1615RGBC-WS2812B"
 			(at 0 2.25 0)
 			(layer "F.Fab")
@@
 			)
 		)
-		(property "Value" "XL-1010RGBC-WS2812B"
+		(property "Value" "XL-1615RGBC-WS2812B"
 			(at 0 2.25 0)
 			(layer "F.Fab")
@@
 			)
 		)
-		(property "Value" "XL-1010RGBC-WS2812B"
+		(property "Value" "XL-2020RGBC-WS2812B"
 			(at 0 2.25 0)
 			(layer "F.Fab")
@@
 			)
 		)
-		(property "Value" "XL-1010RGBC-WS2812B"
+		(property "Value" "XL-2020RGBC-WS2812B"
 			(at 0 2.25 0)
 			(layer "F.Fab")
@@
 			)
 		)
-		(property "Value" "XL-1010RGBC-WS2812B"
+		(property "Value" "XL-2020RGBC-WS2812B"
 			(at 0 2.25 0)
 			(layer "F.Fab")
@@
 			)
 		)
-		(property "Value" "XL-1010RGBC-WS2812B"
+		(property "Value" "XL-2020RGBC-WS2812B"
 			(at 0 2.25 0)
 			(layer "F.Fab")
@@
 			)
 		)
-		(property "Value" "XL-1010RGBC-WS2812B"
+		(property "Value" "XL-2020RGBC-WS2812B"
 			(at 0 2.25 0)
 			(layer "F.Fab")
@@
 			)
 		)
-		(property "Value" "XL-1010RGBC-WS2812B"
+		(property "Value" "XL-2020RGBC-WS2812B"
 			(at 0 2.25 90)
 			(layer "F.Fab")
@@
 			)
 		)
-		(property "Value" "XL-1010RGBC-WS2812B"
+		(property "Value" "XL-2020RGBC-WS2812B"
 			(at 0 2.25 0)
 			(layer "F.Fab")
@@
 			)
 		)
-		(property "Value" "XL-1010RGBC-WS2812B"
+		(property "Value" "XL-1615RGBC-WS2812B"
 			(at 0 2.25 0)
 			(layer "F.Fab")
@@
 			)
 		)
-		(property "Value" "XL-1010RGBC-WS2812B"
+		(property "Value" "XL-2020RGBC-WS2812B"
 			(at 0 2.25 90)
 			(layer "F.Fab")
@@
 			)
 		)
-		(property "Value" "XL-1010RGBC-WS2812B"
+		(property "Value" "XL-1615RGBC-WS2812B"
 			(at 0 2.25 0)
 			(layer "F.Fab")
@@
 			)
 		)
-		(property "Value" "XL-1010RGBC-WS2812B"
+		(property "Value" "XL-2020RGBC-WS2812B"
 			(at 0 2.25 90)
 			(layer "F.Fab")
@@
 			)
 		)
-		(property "Value" "XL-1010RGBC-WS2812B"
+		(property "Value" "XL-2020RGBC-WS2812B"
 			(at 0 2.25 0)
 			(layer "F.Fab")
@@
 			)
 		)
-		(property "Value" "XL-1010RGBC-WS2812B"
+		(property "Value" "XL-2020RGBC-WS2812B"
 			(at 0 2.25 0)
 			(layer "F.Fab")
@@
 			)
 		)
-		(property "Value" "XL-1010RGBC-WS2812B"
+		(property "Value" "XL-2020RGBC-WS2812B"
 			(at 0 2.25 0)
 			(layer "F.Fab")
@@
 			)
 		)
-		(property "Value" "XL-1010RGBC-WS2812B"
+		(property "Value" "XL-1615RGBC-WS2812B"
 			(at 0 2.25 0)
 			(layer "F.Fab")
@@
 			)
 		)
-		(property "Value" "XL-1010RGBC-WS2812B"
+		(property "Value" "XL-1615RGBC-WS2812B"
 			(at 0 2.25 0)
 			(layer "F.Fab")
@@
 			)
 		)
-		(property "Value" "XL-1010RGBC-WS2812B"
+		(property "Value" "XL-2020RGBC-WS2812B"
 			(at 0 2.25 90)
 			(layer "F.Fab")
@@
 			)
 		)
-		(property "Value" "XL-1010RGBC-WS2812B"
+		(property "Value" "XL-1615RGBC-WS2812B"
 			(at 0 2.25 0)
 			(layer "F.Fab")

Commit message: Update test seven seg
Parts:
- added D41: XL-1615RGBC-WS2812B, RevK:SMD1615, F.Cu at (97.8, 97.7)
- added D42: XL-1615RGBC-WS2812B, RevK:SMD1615, F.Cu at (95.7, 103.7)
- added D43: XL-1615RGBC-WS2812B, RevK:SMD1615, F.Cu at (99.8, 105.8)
- added D44: XL-1615RGBC-WS2812B, RevK:SMD1615, F.Cu at (97.8, 103.7)
- added D45: XL-1615RGBC-WS2812B, RevK:SMD1615, F.Cu at (99.8, 103.7)
- added D46: XL-1615RGBC-WS2812B, RevK:SMD1615, F.Cu at (97.8, 95.9)
- added D47: XL-1615RGBC-WS2812B, RevK:SMD1615, F.Cu at (97.8, 94.1)
- added D48: XL-1615RGBC-WS2812B, RevK:SMD1615, F.Cu at (97.8, 92.3)
- moved D20 11.8 mm to (99.8, 107.9)
- moved D17 8.61 mm to (99.8, 110.0)
- moved D18 8.01 mm to (97.8, 107.9)
- moved D19 7.91 mm to (95.7, 105.8)
- moved D15 5.81 mm to (97.8, 99.5)
- moved D14 5.50 mm to (99.8, 112.1)
- moved D16 4.75 mm to (95.7, 107.9)
- moved D13 2.11 mm to (95.7, 110.0)
- moved D1 2.10 mm to (90.4, 112.5)
- moved D10 2.10 mm to (90.4, 94.5)
- moved D2 2.10 mm to (90.4, 110.5)
- moved D3 2.10 mm to (90.4, 108.5)
- moved D4 2.10 mm to (90.4, 106.5)
- moved D5 2.10 mm to (90.4, 104.5)
- moved D6 2.10 mm to (90.4, 102.5)
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Connections:
- D15 pad 2: Net-(D14-O) -> Net-(D15-I)
- D16 pad 2: Net-(D15-O) -> Net-(D14-O)
- D20 pad 4: unconnected-(D20-O-Pad4) -> Net-(D20-O)
Routing:
- net +3V3: track 32.6 -> 111.3 mm
- net Net-(D42-O): track 0.00 -> 10.2 mm, vias 0 -> 2
- net Net-(D16-O): track 1.60 -> 10.4 mm, vias 0 -> 2
- net Net-(D19-O): track 1.60 -> 10.2 mm, vias 0 -> 2
- net Net-(D13-O): track 1.60 -> 10.1 mm, vias 0 -> 2
- net Net-(D44-O): track 0.00 -> 6.85 mm, vias 0 -> 2
- net Net-(D11-O): track 1.60 -> 8.06 mm, vias 0 -> 2
- net Net-(D20-O): track 0.00 -> 4.35 mm
- net Net-(D15-I): track 0.00 -> 4.16 mm, vias 0 -> 2
- net Net-(D14-O): track 1.60 -> 4.03 mm
- net Net-(D46-O): track 0.00 -> 1.60 mm
- net Net-(D41-O): track 0.00 -> 1.60 mm
- net Net-(D47-O): track 0.00 -> 1.60 mm
- net Net-(D43-O): track 0.00 -> 1.06 mm
- net Net-(D11-I): track 4.78 -> 5.41 mm
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
Commit message: Tweak board
Parts:
- added TP10: TestPoint, RevK:PAD-2mm, F.Cu at (109.1, 120.5)
- added TP6: TestPoint, RevK:PAD-2mm, F.Cu at (89.4, 91.7)
- added TP7: TestPoint, RevK:PAD-2mm, F.Cu at (95.0, 91.8)
- added TP8: TestPoint, RevK:PAD-2mm, F.Cu at (101.4, 89.1)
- added TP9: TestPoint, RevK:PAD-2mm, F.Cu at (107.7, 89.1)
- moved D14 0.10 mm to (99.9, 112.1)
- moved D17 0.10 mm to (99.9, 110.0)
- moved D20 0.10 mm to (99.9, 107.9)
- moved D43 0.10 mm to (99.9, 105.8)
- moved D45 0.10 mm to (99.9, 103.7)
Connections:
- D10 pad 1: unconnected-(D10-O-Pad1) -> Net-(D10-O)
- D30 pad 1: unconnected-(D30-O-Pad1) -> Net-(D30-O)
- D40 pad 1: unconnected-(D40-O-Pad1) -> Net-(D40-O)
- D48 pad 4: unconnected-(D48-O-Pad4) -> Net-(D48-O)
Routing:
- net +3V3: track 111.3 -> 68.0 mm
- net Net-(D40-O): track 0.00 -> 3.73 mm
- net Net-(D10-O): track 0.00 -> 2.97 mm
- net Net-(D48-O): track 0.00 -> 2.19 mm
- net Net-(D30-O): track 0.00 -> 2.17 mm
- net GND: vias 1 -> 6

Commit message: Library update
Parts:
- moved D45 0.22 mm to (99.8, 103.9)
- moved D42 0.22 mm to (95.8, 103.9)
- moved D14 0.22 mm to (99.8, 111.9)
- moved D11 0.22 mm to (95.8, 111.9)
- moved D44 0.20 mm to (97.8, 103.9)
- moved D12 0.20 mm to (97.8, 111.9)
- moved D43 0.14 mm to (99.8, 105.9)
- moved D17 0.14 mm to (99.8, 109.9)
- moved D19 0.14 mm to (95.8, 105.9)
- moved D13 0.14 mm to (95.8, 109.9)
- moved D20 0.10 mm to (99.8, 107.9)
- moved D16 0.10 mm to (95.8, 107.9)
