File: PCB/LEDX12/LED.kicad_pcb (KiCad board)
At the start: 2 copper layers, 70 x 70 mm, 33 parts, among them J1 Conn_01x03, J2 TC2030-USB-NL-DS, P1 Square, P2 Square, P3 Square, P4 Square, U1 TPS562246, U2 ESP32-S3-MINI-1, U3 ICS43434_MEMS_Mic

Commit message: Update test seven seg
Parts:
- U2: value ESP32-S3-MINI-1 -> ESP32-S3-MINI-1-N4R2

Commit message: Library update
Parts:
- added D6: MBR0530, RevK:D_SOD-123, B.Cu at (108.2, 106.8)
- moved C12 4.25 mm to (97.4, 106.9)
- moved C16 4.25 mm to (100.0, 106.9)
- moved C2 4.25 mm to (102.5, 107.0)
Connections:
- C1 pad 1: DC -> Net-(D6-A)
- C12 pad 1: DC -> Net-(D6-A)
- C16 pad 1: DC -> Net-(D6-A)
- C2 pad 1: DC -> Net-(D6-A)
- J1 pad 3: DC -> Net-(D6-A)
Routing:
- net Net-(D6-A): track 0.00 -> 24.7 mm
- net DC: track 42.4 -> 19.8 mm
Other:
- board text added: "5V- 17V"
- board text added: "China"
- board text removed: "5-17V"
- board text removed: "Made in China"
