File: PCB/30x9/30x9.kicad_pcb (KiCad board)
At the start: 2 copper layers, 76.2 x 22.9 mm, 508 parts

Commit message: Re render
Parts:
- added TP7: TestPoint, RevK:PAD-2mm, B.Cu at (133.3, 86.4)
- added TP9: TestPoint, RevK:PAD-2mm, B.Cu at (133.3, 91.4)
Routing:
- net Net-(D135-O): track 22.9 -> 24.8 mm
Other:
- board text added: "${CURRENT_DATE}"
- board text added: "+"
- board text added: "-"
- board text added: "3.3V-5V"
- board text added: "A"
- board text added: "I"
- board text added: "Made in China for Andrews&Arnold Ltd"
- board text added: "O"
