File: PCB/30x9/30x9.kicad_sch (KiCad schematic)
At the start: 508 parts

Commit message: Re render
Parts:
- added TP7, TP9: TestPoint, RevK:PAD-2mm, symbol Connector:TestPoint
Connections:
- net GND: now also TP7.1
- net VCC: now also TP9.1
